Commit message: Created launch file, debugging urdf not showing in rviz

File: pf400_description/urdf/PF3400SX.urdf (robot description, URDF)
Before this commit: robot PF3400SX Robot, 7 links, 6 joints
Links:
- link hand: geometry visual mesh filename=package://pf400_description/meshes/PF3400_Hand.STL scale=0.001 0.001 0.001
- link inner_link: geometry visual mesh filename=package://pf400_description/meshes/PF3400_Inner_Link.STL scale=0.001 0.001 0.001
- link left_finger: geometry visual mesh filename=package://pf400_description/meshes/PF3400_Left_Finger.STL scale=0.001 0.001 0.001
- link outer_link: geometry visual mesh filename=package://pf400_description/meshes/PF3400_Outer_Link.STL scale=0.001 0.001 0.001
- link right_finger: geometry visual mesh filename=package://pf400_description/meshes/PF3400_Right_Finger.STL scale=0.001 0.001 0.001
- link z_carriage: geometry visual mesh filename=package://pf400_description/meshes/PF3400_Z_Carriage.STL scale=0.001 0.001 0.001
- link z_column: geometry visual mesh filename=package://pf400_description/meshes/PF3400_Z_Column.STL scale=0.001 0.001 0.001

Commit message: Fixing description launch files

File: pf400_description/urdf/PF3400SX.urdf (robot description, URDF)
Before this commit: robot PF3400SX Robot, 7 links, 6 joints
Links:
- link z_column: geometry visual mesh filename=package://pf400_description/meshes/PF3400_Z_Column.STL scale=0.001 0.001 0.0021
Joints:
- joint J1: limit lower=0.0015 upper=0.4015 effort=1000.0 velocity=0.5 -> lower=0.0015 upper=2.02 effort=1000.0 velocity=0.5
