Commit message: PF400 urdf is fixed and robot now spawns in Rviz

File: pf400_description/urdf/PF400.urdf (robot description, URDF)
Before this commit: robot PF3400SX Robot, 7 links, 6 joints
Links:
- added link base_link; visual mesh filename=package://pf400_description/meshes/base_link.STL scale=1 1 1
- added link rail; visual mesh filename=package://pf400_description/meshes/rail.STL scale=1 1 1
- link z_column: geometry visual mesh filename=package://pf400_description/meshes/PF3400_Z_Column.STL scale=0.001 0.001 0.0022
Joints:
- added joint J6: type prismatic, parent base_link, child rail, origin xyz=0 0 0 rpy=0 0 0, axis 1 0 0, limit lower=-1 upper=1 effort=1000.0 velocity=0.5
- added joint rail_link: type fixed, parent rail, child z_column, origin xyz=0.03005 -0.0198 0.05 rpy=0 0 0, axis 0 1 0, limit lower=0 upper=0 effort=1000.0 velocity=0.5

File: pf400_description/urdf/PF400_URDF.urdf (robot description, URDF)
Before this commit: robot PF400_mate lineer_axis, 6 links, 5 joints
Links:
- link base_link: geometry collision mesh filename=package://pf400_description/meshes/base_link.STL; visual mesh filename=package://pf400_description/meshes/base_link.STL
- link end_effector: geometry collision mesh filename=package://pf400_description/meshes/end_effector.STL; visual mesh filename=package://pf400_description/meshes/end_effector.STL
- link inner_link: geometry collision mesh filename=package://pf400_description/meshes/inner_link.STL; visual mesh filename=package://pf400_description/meshes/inner_link.STL
- link outer_link: geometry collision mesh filename=package://pf400_description/meshes/outer_link.STL; visual mesh filename=package://pf400_description/meshes/outer_link.STL
- link rail: geometry collision mesh filename=package://pf400_description/meshes/rail.STL; visual mesh filename=package://pf400_description/meshes/rail.STL
- link tower: geometry collision mesh filename=package://pf400_description/meshes/tower.STL; visual mesh filename=package://pf400_description/meshes/tower.STL

Commit message: Tower scale is fixed

File: pf400_description/urdf/PF400.urdf (robot description, URDF)
Before this commit: robot PF3400SX Robot, 9 links, 8 joints
Links:
- link z_column: geometry visual mesh filename=package://pf400_description/meshes/PF3400_Z_Column.STL scale=0.001 0.001 0.00132
Joints:
- joint J1: limit lower=0.0015 upper=2.02 effort=1000.0 velocity=0.5 -> lower=0.002 upper=1.12 effort=1000.0 velocity=0.5

Commit message: Adding new finger meshes

File: pf400_description/urdf/PF400.urdf (robot description, URDF)
Before this commit: robot PF3400SX Robot, 9 links, 8 joints
Links:
- link left_finger: geometry visual mesh filename=package://pf400_description/meshes/pf400_left_finger.STL scale=0.001 0.001 0.001
- link right_finger: geometry visual mesh filename=package://pf400_description/meshes/pf400_right_finger.STL scale=0.001 0.001 0.001

Commit message: Description client can now use real robot joint feedback

File: pf400_description/urdf/PF400.urdf (robot description, URDF)
Before this commit: robot PF3400SX Robot, 9 links, 8 joints
Links:
- link hand: geometry visual mesh filename=package://pf400_description/meshes/PF400_Hand.STL scale=0.001 0.001 0.001
- link inner_link: geometry visual mesh filename=package://pf400_description/meshes/PF400_Inner_Link.STL scale=0.001 0.001 0.001
- link outer_link: geometry visual mesh filename=package://pf400_description/meshes/PF400_Outer_Link.STL scale=0.001 0.001 0.001
- link z_carriage: geometry visual mesh filename=package://pf400_description/meshes/PF400_Z_Carriage.STL scale=0.001 0.001 0.001
- link z_column: geometry visual mesh filename=package://pf400_description/meshes/PF400_Z_Column.STL scale=0.001 0.001 0.00132
Joints:
- joint J1: limit lower=0.002 upper=1.12 effort=1000.0 velocity=0.5 -> lower=0.002 upper=1.160 effort=1000.0 velocity=0.5
- joint J2: origin xyz=0.173001 0.020 .0235 rpy=0 0 0 -> xyz=0.173001 0.020 0.0235 rpy=0 0 0
- joint J3: limit lower=0.20944 upper=6.07375 effort=1000.0 velocity=0.5 -> lower=0.175 upper=6.1 effort=1000.0 velocity=0.5
- joint J5: limit lower=0.051954 upper=0.070 effort=1000.0 velocity=0.5 -> lower=0.067454 upper=0.070 effort=1000.0 velocity=0.5
- joint J5_mirror: limit lower=0.051954 upper=0.070 effort=1000.0 velocity=0.5 -> lower=0.067454 upper=0.070 effort=1000.0 velocity=0.5
