Commit message: Working on module urdf

File: pf400_description/urdf/PF400_module.urdf (robot description, URDF)
Before this commit: robot PF3400SX Robot, 9 links, 8 joints
Links:
- added link pf400_module; visual mesh filename=package://pf400_description/meshes/pf400_module.STL scale=1 1 1
Joints:
- added joint Module_table: type fixed, parent pf400_module, child rail_base, origin xyz=0 0 0 rpy=0 0 0, axis 0 0 1, limit lower=0 upper=0 effort=1000.0 velocity=0.5

Commit message: Fixing link tree in URDF

File: pf400_description/urdf/PF400_module.urdf (robot description, URDF)
Before this commit: robot PF3400SX Robot, 10 links, 9 joints
Joints:
- removed joint Module_table
- added joint module_table: type fixed, parent pf400_module, child rail_base, origin xyz=0 0 0 rpy=0 0 0, axis 0 0 1, limit lower=0 upper=0 effort=1000.0 velocity=0.5

Commit message: pf400 module urdf is added

File: pf400_description/urdf/PF400_module.urdf (robot description, URDF)
Before this commit: robot PF3400SX Robot, 10 links, 9 joints
Links:
- link pf400_module: geometry visual mesh filename=package://pf400_description/meshes/PF400_module.STL scale=0.0008 0.0008 0.0008

Commit message: Adding module carts into URDF

File: pf400_description/urdf/PF400_module.urdf (robot description, URDF)
Before this commit: robot PF3400SX Robot, 10 links, 9 joints
Links:
- added link module_cart_link_1; visual mesh filename=package://pf400_description/meshes/module_cart.stl scale=1 1 1
- added link module_cart_link_2; visual mesh filename=package://pf400_description/meshes/module_cart.stl scale=1 1 1
- added link module_cart_link_3; visual mesh filename=package://pf400_description/meshes/module_cart.stl scale=1 1 1
- added link module_cart_link_4; visual mesh filename=package://pf400_description/meshes/module_cart.stl scale=1 1 1
- link pf400_module: geometry visual mesh filename=package://pf400_description/meshes/PF400_module.STL scale=0.001 0.001 0.001
Joints:
- added joint module_cart_link_1: type fixed, parent module_cart_link_1, child pf400_module, origin xyz=0 0 0 rpy=0 0 0, axis 0 0 1, limit lower=0 upper=0 effort=1000.0 velocity=0.5
- added joint module_cart_link_2: type fixed, parent module_cart_link_2, child module_cart_link_1, origin xyz=0 0 0 rpy=0 0 0, axis 0 0 1, limit lower=0 upper=0 effort=1000.0 velocity=0.5
- added joint module_cart_link_3: type fixed, parent module_cart_link_3, child module_cart_link_2, origin xyz=0 0 0 rpy=0 0 0, axis 0 0 1, limit lower=0 upper=0 effort=1000.0 velocity=0.5
- added joint module_cart_link_4: type fixed, parent module_cart_link_4, child module_cart_link_3, origin xyz=0 0 0 rpy=0 0 0, axis 0 0 1, limit lower=0 upper=0 effort=1000.0 velocity=0.5

Commit message: Module carts are added to URDF

File: pf400_description/urdf/PF400_module.urdf (robot description, URDF)
Before this commit: robot PF3400SX Robot, 14 links, 13 joints
Links:
- added link module_cart_link_5; visual mesh filename=package://pf400_description/meshes/module_cart.stl scale=1 1 1
- added link module_cart_link_6; visual mesh filename=package://pf400_description/meshes/module_cart.stl scale=1 1 1
- added link module_cart_link_7; visual mesh filename=package://pf400_description/meshes/module_cart.stl scale=1 1 1
- added link module_cart_link_8; visual mesh filename=package://pf400_description/meshes/module_cart.stl scale=1 1 1
Joints:
- added joint module_cart_link_5: type fixed, parent module_cart_link_5, child module_cart_link_4, origin xyz=0 0 0 rpy=0 0 0, axis 0 0 1, limit lower=0 upper=0 effort=1000.0 velocity=0.5
- added joint module_cart_link_6: type fixed, parent module_cart_link_6, child module_cart_link_5, origin xyz=0 0 0 rpy=0 0 0, axis 0 0 1, limit lower=0 upper=0 effort=1000.0 velocity=0.5
- added joint module_cart_link_7: type fixed, parent module_cart_link_7, child module_cart_link_6, origin xyz=0 0 0 rpy=0 0 0, axis 0 0 1, limit lower=0 upper=0 effort=1000.0 velocity=0.5
- added joint module_cart_link_8: type fixed, parent module_cart_link_8, child module_cart_link_7, origin xyz=0 0 0 rpy=0 0 0, axis 0 0 1, limit lower=0 upper=0 effort=1000.0 velocity=0.5

Commit message: Adding OT2 into meshes and urdf

File: pf400_description/urdf/PF400_module.urdf (robot description, URDF)
Before this commit: robot PF3400SX Robot, 18 links, 17 joints
Links:
- added link OT2; visual mesh filename=package://pf400_description/meshes/OT2.STL scale=1 1 1
Joints:
- added joint OT2: type fixed, parent module_cart_link_2, child OT2, origin xyz=0 0 0 rpy=0 0 0, axis 0 0 1, limit lower=0 upper=0 effort=1000.0 velocity=0.5

Commit message: Fixing OT2 scale

File: pf400_description/urdf/PF400_module.urdf (robot description, URDF)
Before this commit: robot PF3400SX Robot, 19 links, 18 joints
Links:
- link OT2: geometry visual mesh filename=package://pf400_description/meshes/OT2.STL scale=0.001 0.001 0.001

Commit message: Adde 2 OT2 into URDF

File: pf400_description/urdf/PF400_module.urdf (robot description, URDF)
Before this commit: robot PF3400SX Robot, 19 links, 18 joints
Links:
- added link OT2_2; visual mesh filename=package://pf400_description/meshes/OT2.STL scale=0.001 0.001 0.001
Joints:
- added joint OT2_2: type fixed, parent OT2, child OT2_2, origin xyz=0 0 0 rpy=0 0 0, axis 0 0 1, limit lower=0 upper=0 effort=1000.0 velocity=0.5
