Commit message: Fixed gripper hight

File: pf400_description/urdf/pcr_workcell.urdf (robot description, URDF)
Before this commit: robot PF3400SX Robot, 20 links, 19 joints
Joints:
- joint J5: limit lower=0.067454 upper=0.070 effort=1000.0 velocity=0.5 -> lower=0.04 upper=0.0675 effort=1000.0 velocity=0.5
- joint J5_mirror: limit lower=0.067454 upper=0.070 effort=1000.0 velocity=0.5 -> lower=0.04 upper=0.0675 effort=1000.0 velocity=0.5

Commit message: Working on OT2 pipette

File: pf400_description/urdf/pcr_workcell.urdf (robot description, URDF)
Before this commit: robot PCR Workcell, 20 links, 19 joints
Links:
- added link OT2_pipette_base; visual mesh filename=package://pf400_description/meshes/ot2_pipette_base.STL scale=0.001 0.001 0.001
- link OT2: geometry visual mesh filename=package://pf400_description/meshes/OT_2_without_pipette.STL scale=0.001 0.001 0.001
- link OT2_2: geometry visual mesh filename=package://pf400_description/meshes/OT_2_without_pipette.STL scale=0.001 0.001 0.001
Joints:
- added joint pipette_rail_x: type floating, parent OT2, child OT2_pipette_base, origin xyz=0 0 0 rpy=0 0 0, axis -1 -1 0, limit lower=0 upper=0.2 effort=1000.0 velocity=0.5

Commit message: Working on OT2 pipette joints

File: pf400_description/urdf/pcr_workcell.urdf (robot description, URDF)
Before this commit: robot PCR Workcell, 21 links, 20 joints
Links:
- added link OT2_pipette; visual mesh filename=package://pf400_description/meshes/pipette.STL scale=0.001 0.001 0.001
- added link OT2_pipette_rail; visual mesh filename=package://pf400_description/meshes/ot2_pipette_base.STL scale=0.001 0.001 0.001
Joints:
- added joint pipette: type prismatic, parent OT2_pipette_base, child OT2_pipette, origin xyz=0 0 0 rpy=0 0 0, axis 0 0 -1, limit lower=0 upper=0.06 effort=1000.0 velocity=0.5
- added joint pipette_rail_y: type prismatic, parent OT2, child OT2_pipette_rail, origin xyz=0 0 0 rpy=0 0 0, axis 0 -1 0, limit lower=0 upper=0.3 effort=1000.0 velocity=0.5
- joint pipette_rail_x: axis -1 -1 0 -> -1 0 0; limit lower=0 upper=0.2 effort=1000.0 velocity=0.5 -> lower=0 upper=0.3 effort=1000.0 velocity=0.5; parent OT2 -> OT2_pipette_rail; type floating -> prismatic

Commit message: Changing pipette rail stl file

File: pf400_description/urdf/pcr_workcell.urdf (robot description, URDF)
Before this commit: robot PCR Workcell, 23 links, 22 joints
Links:
- link OT2_pipette_rail: geometry visual mesh filename=package://pf400_description/meshes/ot2_pipette_rail.STL scale=0.001 0.001 0.001

Commit message: Added new OT2 description

File: pf400_description/urdf/pcr_workcell.urdf (robot description, URDF)
Before this commit: robot PCR Workcell, 23 links, 22 joints
Links:
- removed link OT2_pipette
- added link OT2_8_channel_pipette; visual mesh filename=package://pf400_description/meshes/OT2_8ch_pipette.stl scale=1 1 1
- added link OT2_single_pipette; visual mesh filename=package://pf400_description/meshes/pipette.STL scale=0.001 0.001 0.001
- link OT2: geometry visual mesh filename=package://pf400_description/meshes/OT2_base.stl scale=1 1 1
- link OT2_pipette_base: geometry visual mesh filename=package://pf400_description/meshes/OT2_pipette_base.stl scale=1 1 1
- link OT2_pipette_rail: geometry visual mesh filename=package://pf400_description/meshes/OT2_rail.stl scale=1 1 1
Joints:
- removed joint pipette
- added joint 8_channel_pipette: type prismatic, parent OT2_pipette_base, child OT2_8_channel_pipette, origin xyz=0 0 0 rpy=0 0 0, axis 0 0 -1, limit lower=0 upper=0.18 effort=1000.0 velocity=0.5
- added joint single_pipette: type prismatic, parent OT2_pipette_base, child OT2_single_pipette, origin xyz=0 0 0 rpy=0 0 0, axis 0 0 -1, limit lower=0 upper=0.18 effort=1000.0 velocity=0.5

Commit message: Adding Thermocycler description

File: pf400_description/urdf/pcr_workcell.urdf (robot description, URDF)
Before this commit: robot PCR Workcell, 24 links, 23 joints
Links:
- added link Thermocycler_Base; visual mesh filename=package://pf400_description/meshes/thermocycler_base.stl scale=1 1 1
- added link Thermocycler_Cap; visual mesh filename=package://pf400_description/meshes/thermocycler_cap.stl scale=1 1 1
Joints:
- added joint Thermocycler_Base: type fixed, parent module_cart_link_4, child Thermocycler_Base, origin xyz=0 0 0 rpy=0 0 0, axis 0 0 1, limit lower=0 upper=0 effort=1000.0 velocity=0.5
- added joint Thermocycler_Cap: type fixed, parent Thermocycler_Base, child Thermocycler_Cap, origin xyz=0 0 0 rpy=0 0 0, axis 0 0 1, limit lower=0 upper=1 effort=1000.0 velocity=0.5

Commit message: Fixed thermocycler description

File: pf400_description/urdf/pcr_workcell.urdf (robot description, URDF)
Before this commit: robot PCR Workcell, 26 links, 25 joints
Links:
- link Thermocycler_Base: geometry visual mesh filename=package://pf400_description/meshes/thermocycler_base.STL scale=0.001 0.001 0.001
- link Thermocycler_Cap: geometry visual mesh filename=package://pf400_description/meshes/thermocycler_cap.STL scale=0.001 0.001 0.001
Joints:
- joint Thermocycler_Base: origin xyz=0 0 0 rpy=0 0 0 -> xyz=-0.2 0.2 0 rpy=0 0 0
- joint Thermocycler_Cap: axis 0 0 1 -> -1 0 0; limit lower=0 upper=1 effort=1000.0 velocity=0.5 -> lower=0 upper=1.2 effort=1000.0 velocity=0.5; origin xyz=0 0 0 rpy=0 0 0 -> xyz=0 0.466 1.05 rpy=1.5708 0 0; type fixed -> revolute

Commit message: Added peeler and sealer into urdf

File: pf400_description/urdf/pcr_workcell.urdf (robot description, URDF)
Before this commit: robot PCR Workcell, 26 links, 25 joints
Links:
- added link Peeler_Base; visual mesh filename=package://pf400_description/meshes/peeler_base.STL scale=0.001 0.001 0.001
- added link Peeler_Plate; visual mesh filename=package://pf400_description/meshes/peeler_plate.STL scale=0.001 0.001 0.001
- added link Sealer_Base; visual mesh filename=package://pf400_description/meshes/sealer_base.STL scale=0.001 0.001 0.001
- added link Sealer_Plate; visual mesh filename=package://pf400_description/meshes/sealer_plate.STL scale=0.001 0.001 0.001
Joints:
- added joint Peeler_Base: type fixed, parent module_cart_link_5, child Peeler_Base, origin xyz=1.15 -0.37 1.042 rpy=0 0 0, axis 0 0 0, limit lower=0 upper=0 effort=1000.0 velocity=0.5
- added joint Peeler_Plate: type prismatic, parent Peeler_Base, child Peeler_Plate, origin xyz=0.23 -0.03 0.083 rpy=1.5708 0 0, axis 0 0 1, limit lower=0 upper=0.3 effort=1000.0 velocity=0.5
- added joint Sealer_Base: type fixed, parent module_cart_link_5, child Sealer_Base, origin xyz=-0.2 0.2 0 rpy=0 0 0, axis 0 0 1, limit lower=0 upper=0 effort=1000.0 velocity=0.5
- added joint Sealer_Plate: type prismatic, parent Sealer_Base, child Sealer_Plate, origin xyz=0 0.466 1.05 rpy=1.5708 0 0, axis 0 0 1, limit lower=0 upper=0.25 effort=1000.0 velocity=0.5

Commit message: Fixing peeler origin

File: pf400_description/urdf/pcr_workcell.urdf (robot description, URDF)
Before this commit: robot PCR Workcell, 30 links, 29 joints
Joints:
- joint Sealer_Base: origin xyz=-0.2 0.2 0 rpy=0 0 0 -> xyz=1.55 -1.05 1.042 rpy=0 0 0
- joint Sealer_Plate: origin xyz=0 0.466 1.05 rpy=1.5708 0 0 -> xyz=0.045 0.28 0.01 rpy=1.5708 0 0

Commit message: Fixing Sealer origin

File: pf400_description/urdf/pcr_workcell.urdf (robot description, URDF)
Before this commit: robot PCR Workcell, 30 links, 29 joints
Joints:
- joint Sealer_Plate: origin xyz=0.045 0.28 0.01 rpy=1.5708 0 0 -> xyz=0.057 0.28 0.01 rpy=1.5708 0 0
