Commit message: Fixed the module cart locations

File: pf400_description/urdf/materials.xacro (robot description, xacro)
@@ -44,5 +44,5 @@
   </material>
   <material name="darkbluegreen" >
-    <color rgba="0.0 0.1 0.13 1.0" />
+    <color rgba="0.0 0.2 0.23 1.0" />
   </material>
   <material name="aluminum">

File: pf400_description/urdf/module_carts.urdf.xacro (robot description, xacro)
@@ -5,5 +5,5 @@
   <link name="${prefix}cart_1">
     <visual>
-      <origin xyz="1.32 0.847 0" rpy="0 0 0"/>
+      <origin xyz="0 0 0" rpy="0 0 0"/>
       <geometry>
         <mesh filename="package://pf400_description/meshes/module_cart.stl" scale="1 1 1"/>
@@ -14,5 +14,5 @@
   <link name="${prefix}cart_2">
     <visual>
-      <origin xyz="0.51 0.847 0" rpy="0 0 0"/>
+      <origin xyz="0 0 0" rpy="0 0 0"/>
       <geometry>
         <mesh filename="package://pf400_description/meshes/module_cart.stl" scale="1 1 1"/>
@@ -23,5 +23,5 @@
   <link name="${prefix}cart_3">
     <visual>
-      <origin xyz="-0.368 0.847 0" rpy="0 0 0"/>
+      <origin xyz="0 0 0" rpy="0 0 0"/>
       <geometry>
         <mesh filename="package://pf400_description/meshes/module_cart.stl" scale="1 1 1"/>
@@ -32,5 +32,5 @@
   <link name="${prefix}cart_4">
     <visual>
-      <origin xyz="-1.18 0.847 0" rpy="0 0 0"/>
+      <origin xyz="0 0 0" rpy="0 0 0"/>
       <geometry>
         <mesh filename="package://pf400_description/meshes/module_cart.stl" scale="1 1 1"/>
@@ -41,5 +41,5 @@
   <link name="${prefix}cart_5">
     <visual>
-      <origin xyz="1.32  -0.548 0" rpy="0 0 0"/>
+      <origin xyz="0 0 0" rpy="0 0 0"/>
       <geometry>
         <mesh filename="package://pf400_description/meshes/module_cart.stl" scale="1 1 1"/>
@@ -50,5 +50,5 @@
   <link name="${prefix}cart_6">
     <visual>
-      <origin xyz="0.51 -0.548 0" rpy="0 0 0"/>
+      <origin xyz="0 0 0" rpy="0 0 0"/>
       <geometry>
         <mesh filename="package://pf400_description/meshes/module_cart.stl" scale="1 1 1"/>
@@ -59,5 +59,5 @@
   <link name="${prefix}cart_7">
     <visual>
-      <origin xyz="-0.368 -0.548 0" rpy="0 0 0"/>
+      <origin xyz="0 0 0" rpy="0 0 0"/>
       <geometry>
         <mesh filename="package://pf400_description/meshes/module_cart.stl" scale="1 1 1"/>
@@ -68,5 +68,5 @@
   <link name="${prefix}cart_8">
     <visual>
-      <origin xyz="-1.18 -0.548 0" rpy="0 0 0"/>
+      <origin xyz="0 0 0" rpy="0 0 0"/>
       <geometry>
         <mesh filename="package://pf400_description/meshes/module_cart.stl" scale="1 1 1"/>
@@ -86,57 +86,57 @@
   <!-- Joints -->
   <joint name="pf400_cart_to_cart_1" type="fixed">
-    <parent link="${prefix}cart_1"/>
-    <child link="${prefix}pf400_cart"/>
+    <parent link="${prefix}pf400_cart"/>
+    <child link="${prefix}cart_1"/>
     <axis xyz="0 0 1"/>
-    <origin xyz="0 0 0" rpy="0 0 0"/>
+    <origin xyz="0.99 0.806 0" rpy="0 0 0"/>
     <limit effort="1000.0" lower="0" upper="0" velocity="0.5"/>
   </joint>
-  <joint name="cart_1_to_cart_2" type="fixed">
-    <parent link="${prefix}cart_2"/>
-    <child link="${prefix}cart_1"/>
+  <joint name="pf400_cart_to_cart_2" type="fixed">
+    <parent link="${prefix}pf400_cart"/>
+    <child link="${prefix}cart_2"/>
     <axis xyz="0 0 1"/>
-    <origin xyz="0 0 0" rpy="0 0 0"/>
+    <origin xyz="0.24 0.806 0" rpy="0 0 0"/>
     <limit effort="1000.0" lower="0" upper="0" velocity="0.5"/>
   </joint>
-  <joint name="cart_2_to_cart_3" type="fixed">
-    <parent link="${prefix}cart_3"/>
-    <child link="${prefix}cart_2"/>
+  <joint name="pf400_cart_to_cart_3" type="fixed">
+    <parent link="${prefix}pf400_cart"/>
+    <child link="${prefix}cart_3"/>
     <axis xyz="0 0 1"/>
-    <origin xyz="0 0 0" rpy="0 0 0"/>
+    <origin xyz="-0.51 0.806  0" rpy="0 0 0"/>
     <limit effort="1000.0" lower="0" upper="0" velocity="0.5"/>
   </joint>
-  <joint name="cart_3_to_cart_4" type="fixed">
-    <parent link="${prefix}cart_4"/>
-    <child link="${prefix}cart_3"/>
+  <joint name="pf400_cart_to_cart_4" type="fixed">
+    <parent link="${prefix}pf400_cart"/>
+    <child link="${prefix}cart_4"/>
     <axis xyz="0 0 1"/>
-    <origin xyz="0 0 0" rpy="0 0 0"/>
+    <origin xyz="-1.26 0.806  0" rpy="0 0 0"/>
     <limit effort="1000.0" lower="0" upper="0" velocity="0.5"/>
   </joint>
-  <joint name="cart_4_to_cart_5" type="fixed">
-    <parent link="${prefix}cart_5"/>
-    <child link="${prefix}cart_4"/>
+  <joint name="pf400_cart_to_cart_5" type="fixed">
+    <parent link="${prefix}pf400_cart"/>
+    <child link="${prefix}cart_5"/>
     <axis xyz="0 0 1"/>
-    <origin xyz="0 0 0" rpy="0 0 0"/>
+    <origin xyz="0.99 -0.451 0" rpy="0 0 0"/>
     <limit effort="1000.0" lower="0" upper="0" velocity="0.5"/>
   </joint>
-  <joint name="cart_5_to_cart_6" type="fixed">
-    <parent link="${prefix}cart_6"/>
-    <child link="${prefix}cart_5"/>
+  <joint name="pf400_cart_to_cart_6" type="fixed">
+    <parent link="${prefix}pf400_cart"/>
+    <child link="${prefix}cart_6"/>
     <axis xyz="0 0 1"/>
-    <origin xyz="0 0 0" rpy="0 0 0"/>
+    <origin xyz="0.24 -0.451 0" rpy="0 0 0"/>
     <limit effort="1000.0" lower="0" upper="0" velocity="0.5"/>
   </joint>
-  <joint name="cart_6_to_cart_7" type="fixed">
-    <parent link="${prefix}cart_7"/>
-    <child link="${prefix}cart_6"/>
+  <joint name="pf400_cart_to_cart_7" type="fixed">
+    <parent link="${prefix}pf400_cart"/>
+    <child link="${prefix}cart_7"/>
     <axis xyz="0 0 1"/>
-    <origin xyz="0 0 0" rpy="0 0 0"/>
+    <origin xyz="-0.51 -0.451 0" rpy="0 0 0"/>
     <limit effort="1000.0" lower="0" upper="0" velocity="0.5"/>
   </joint>
-  <joint name="cart_7_to_cart_8" type="fixed">
-    <parent link="${prefix}cart_8"/>
-    <child link="${prefix}cart_7"/>
+  <joint name="pf400_cart_to_cart_8" type="fixed">
+    <parent link="${prefix}pf400_cart"/>
+    <child link="${prefix}cart_8"/>
     <axis xyz="0 0 1"/>
-    <origin xyz="0 0 0" rpy="0 0 0"/>
+    <origin xyz="-1.26 -0.451 0" rpy="0 0 0"/>
     <limit effort="1000.0" lower="0" upper="0" velocity="0.5"/>
   </joint>
