Commit message: Fixing the plate oriantation

File: pf400_description/urdf/peeler.urdf.xacro (robot description, xacro)
@@ -14,5 +14,5 @@
   <link name="${prefix}peeler_plate">
     <visual>
-      <origin xyz="0 0 0" rpy="0 0 0"/>
+      <origin xyz="0 0 0" rpy="0 1.5708 0"/>
       <geometry>
         <mesh filename="package://pf400_description/meshes/peeler_plate.STL" scale="0.001 0.001 0.001"/>
@@ -26,5 +26,5 @@
     <child link="${prefix}peeler_plate"/>
     <axis xyz="0 0 1"/>
-    <origin xyz="0.23 -0.03 0.083" rpy="1.5708 0 0"/>
+    <origin xyz="0.25 -0.18 0.083" rpy="1.5708 0 0"/>
     <limit effort="1000.0" lower="0" upper="0.3" velocity="0.5"/>
   </joint>
