Commit message: Clean up

File: pf400_description/urdf/thermocycler.urdf.xacro (robot description, xacro)
@@ -3,5 +3,5 @@
   <!-- Links -->
   <xacro:macro name="Thermocycler" params = "prefix">
-  <link name="${prefix}Thermocycler_Base">
+  <link name="${prefix}thermocycler_base">
     <visual>
       <origin xyz="0 0.5 1.042" rpy="1.5708 0 0"/>
@@ -12,5 +12,5 @@
     </visual>
   </link>
-  <link name="${prefix}Thermocycler_Cap">
+  <link name="${prefix}thermocycler_cap">
     <visual>
       <origin xyz="0 0 0" rpy="0 0 0"/>
@@ -23,6 +23,6 @@
   <!-- Joints -->
   <joint name="Thermocycler_Cap" type="revolute">
-    <parent link="${prefix}Thermocycler_Base"/>
-    <child link="${prefix}Thermocycler_Cap"/>
+    <parent link="${prefix}thermocycler_base"/>
+    <child link="${prefix}thermocycler_cap"/>
     <axis xyz="-1 0 0"/>
     <origin xyz="0 0.466 1.05" rpy="1.5708 0 0"/>

Commit message: Adding the second thermocycler

File: pf400_description/urdf/thermocycler.urdf.xacro (robot description, xacro)
@@ -21,4 +21,22 @@
     </visual>
   </link>
+  <link name="${prefix}thermocycler_base2">
+    <visual>
+      <origin xyz="0 0.5 1.042" rpy="1.5708 0 0"/>
+      <geometry>
+        <mesh filename="package://pf400_description/meshes/thermocycler_base.STL" scale="0.001 0.001 0.001"/>
+      </geometry>
+      <material name="light_grey"/>
+    </visual>
+  </link>
+  <link name="${prefix}thermocycler_cap2">
+    <visual>
+      <origin xyz="0 0 0" rpy="0 0 0"/>
+      <geometry>
+        <mesh filename="package://pf400_description/meshes/thermocycler_cap.STL" scale="0.001 0.001 0.001"/>
+      </geometry>
+      <material name="red"/>
+    </visual>
+  </link>
   <!-- Joints -->
   <joint name="Thermocycler_Cap" type="fixed">
@@ -29,4 +47,11 @@
     <limit effort="1000.0" lower="0" upper="1.2" velocity="0.5"/>
   </joint>
+  <joint name="Thermocycler_Cap2" type="fixed">
+    <parent link="${prefix}thermocycler_base2"/>
+    <child link="${prefix}thermocycler_cap2"/>
+    <axis xyz="-1 0 0"/>
+    <origin xyz="0 0.466 1.05" rpy="1.5708 0 0"/>
+    <limit effort="1000.0" lower="0" upper="1.2" velocity="0.5"/>
+  </joint>
   </xacro:macro>
 </robot>
