Commit message: Individual robot description work

File: pf400_description/urdf/OT2.urdf.xacro (robot description, xacro)
@@ -3,13 +3,4 @@
   <!-- Links -->
   <xacro:macro name="OT2" params = "prefix">
-  <link name="${prefix}rail_base">
-    <visual>
-      <origin xyz="0.125 -0.0198 0" rpy="0 0 1.5708"/>
-      <geometry>
-        <mesh filename="package://pf400_description/meshes/rail_base.STL" scale="1 1 1"/>
-      </geometry>
-      <material name="white"/>
-    </visual>
-  </link>
   <link name="${prefix}OT2">
     <visual>
@@ -48,5 +39,5 @@
     </visual>
   </link>
-  <link name="${prefix}OT2_8_hannel_pipette">
+  <link name="${prefix}OT2_8_channel_pipette">
     <visual>
       <origin xyz="0.51 1.15 1.042" rpy="0 0 0"/>

File: pf400_description/urdf/PF400.urdf.xacro (robot description, xacro)
@@ -90,5 +90,5 @@
     <axis xyz="0 0 1"/>
     <origin xyz="0.03005 -0.0198 0.17535" rpy="0 0 0"/>
-    <limit effort="1000.0" lower="0.002" upper="1.160" velocity="0.5"/>  </joint>
+    <limit effort="1000.0" lower="0.002" upper="1.160" velocity="0.5"/>
   </joint>
   <joint name="J2" type="revolute">

File: pf400_description/urdf/peeler.urdf.xacro (robot description, xacro)
@@ -2,5 +2,5 @@
 <robot name="Peeler" xmlns:xacro="http://www.ros.org/wiki/xacro">
   <!-- Links -->
-  <xacro:macro name="peeler" params = "prefix">
+  <xacro:macro name="Peeler" params = "prefix">
     <link name="${prefix}peeler_base">
     <visual>

Commit message: Fixing initilzation issue

File: pf400_description/urdf/OT2.urdf.xacro (robot description, xacro)
@@ -49,5 +49,5 @@
   </link>
   <!-- Joints -->
-  <joint name="OT2_1_Pipette_Joint1" type="prismatic">
+  <joint name="OT2_1_Pipette_Joint1" type="fixed">
     <parent link="${prefix}OT2"/>
     <child link="${prefix}OT2_pipette_rail"/>
@@ -56,5 +56,5 @@
     <limit effort="1000.0" lower="0" upper="0.3" velocity="0.5"/>
   </joint>
-  <joint name="OT2_1_Pipette_Joint2" type="prismatic">
+  <joint name="OT2_1_Pipette_Joint2" type="fixed">
     <parent link="${prefix}OT2_pipette_rail"/>
     <child link="${prefix}OT2_pipette_base"/>
@@ -63,5 +63,5 @@
     <limit effort="1000.0" lower="0" upper="0.3" velocity="0.5"/>
   </joint>
-  <joint name="OT2_1_Single_Pipette" type="prismatic">
+  <joint name="OT2_1_Single_Pipette" type="fixed">
     <parent link="${prefix}OT2_pipette_base"/>
     <child link="${prefix}OT2_single_pipette"/>
@@ -70,5 +70,5 @@
     <limit effort="1000.0" lower="0" upper="0.18" velocity="0.5"/>
   </joint>
-  <joint name="OT2_1_8_Channel_Pipette" type="prismatic">
+  <joint name="OT2_1_8_Channel_Pipette" type="fixed">
     <parent link="${prefix}OT2_pipette_base"/>
     <child link="${prefix}OT2_8_channel_pipette"/>

File: pf400_description/urdf/peeler.urdf.xacro (robot description, xacro)
@@ -22,5 +22,5 @@
   </link>
   <!-- Joints -->
-  <joint name="Peeler_Plate_Joint" type="prismatic">
+  <joint name="Peeler_Plate_Joint" type="fixed">
     <parent link="${prefix}peeler_base"/>
     <child link="${prefix}peeler_plate"/>

File: pf400_description/urdf/sealer.urdf.xacro (robot description, xacro)
@@ -22,5 +22,5 @@
   </link>
   <!-- Joints -->
-  <joint name="Sealer_Plate_Joint" type="prismatic">
+  <joint name="Sealer_Plate_Joint" type="fixed">
     <parent link="${prefix}sealer_base"/>
     <child link="${prefix}sealer_plate"/>

File: pf400_description/urdf/thermocycler.urdf.xacro (robot description, xacro)
@@ -22,5 +22,5 @@
   </link>
   <!-- Joints -->
-  <joint name="Thermocycler_Cap" type="revolute">
+  <joint name="Thermocycler_Cap" type="fixed">
     <parent link="${prefix}thermocycler_base"/>
     <child link="${prefix}thermocycler_cap"/>

Commit message: Adding OT2 betha

File: pf400_description/urdf/OT2.urdf.xacro (robot description, xacro)
@@ -3,74 +3,207 @@
   <!-- Links -->
   <xacro:macro name="OT2" params = "prefix">
-  <link name="${prefix}OT2">
-    <visual>
-      <origin xyz="0.36 0.94 1.042" rpy="0 0 0"/>
-      <geometry>
-        <mesh filename="package://pf400_description/meshes/OT2_base.stl" scale="1 1 1"/>
-      </geometry>
-      <material name="aluminum"/>
-    </visual>
-  </link>
-  <link name="${prefix}OT2_pipette_rail">
-    <visual>
-      <origin xyz="0.36 1.15 1.042" rpy="0 0 0"/>
-      <geometry>
-        <mesh filename="package://pf400_description/meshes/OT2_rail.stl" scale="1 1 1"/>
-      </geometry>
-      <material name="aluminum"/>
-    </visual>
-  </link>
-  <link name="${prefix}OT2_pipette_base">
-    <visual>
-      <origin xyz="0.51 1.15 1.042" rpy="0 0 0"/>
-      <geometry>
-        <mesh filename="package://pf400_description/meshes/OT2_pipette_base.stl" scale="1 1 1"/>
-      </geometry>
-      <material name="aluminum"/>
-    </visual>
-  </link>
-  <link name="${prefix}OT2_single_pipette">
-    <visual>
-      <origin xyz="0.79 0.76 1.27" rpy="1.5708 0 1.5708"/>
-      <geometry>
-        <mesh filename="package://pf400_description/meshes/pipette.STL" scale="0.001 0.001 0.001"/>
-      </geometry>
-      <material name="black"/>
-    </visual>
-  </link>
-  <link name="${prefix}OT2_8_channel_pipette">
-    <visual>
-      <origin xyz="0.51 1.15 1.042" rpy="0 0 0"/>
-      <geometry>
-        <mesh filename="package://pf400_description/meshes/OT2_8ch_pipette.stl" scale="1 1 1"/>
-      </geometry>
-      <material name="black"/>
-    </visual>
+  <link name="${prefix}OT2_alpha">
+    <visual>
+      <origin xyz="0.36 0.94 1.042" rpy="0 0 0"/>
+      <geometry>
+        <mesh filename="package://pf400_description/meshes/OT2_base.stl" scale="1 1 1"/>
+      </geometry>
+      <material name="aluminum"/>
+    </visual>
+    <collision>
+      <geometry>
+        <mesh filename="package://pf400_description/meshes/OT2_base.stl" scale="1 1 1"/>
+      </geometry>
+      <origin xyz="0.36 0.94 1.042" rpy="0 0 0"/>
+    </collision>
+  </link>
+  <link name="${prefix}OT2_pipette_rail_alpha">
+    <visual>
+      <origin xyz="0.36 1.15 1.042" rpy="0 0 0"/>
+      <geometry>
+        <mesh filename="package://pf400_description/meshes/OT2_rail.stl" scale="1 1 1"/>
+      </geometry>
+      <material name="aluminum"/>
+    </visual>
+    <collision>
+      <geometry>
+        <mesh filename="package://pf400_description/meshes/OT2_rail.stl" scale="1 1 1"/>
+      </geometry>
+      <origin xyz="0.36 1.15 1.042" rpy="0 0 0"/>
+    </collision>
+  </link>
+  <link name="${prefix}OT2_pipette_base_alpha">
+    <visual>
+      <origin xyz="0.51 1.15 1.042" rpy="0 0 0"/>
+      <geometry>
+        <mesh filename="package://pf400_description/meshes/OT2_pipette_base.stl" scale="1 1 1"/>
+      </geometry>
+      <material name="aluminum"/>
+    </visual>
+    <collision>
+      <geometry>
+        <mesh filename="package://pf400_description/meshes/OT2_pipette_base.stl" scale="1 1 1"/>
+      </geometry>
+      <origin xyz="0.51 1.15 1.042" rpy="0 0 0"/>
+    </collision>
+  </link>
+  <link name="${prefix}OT2_single_pipette_alpha">
+    <visual>
+      <origin xyz="0.79 0.76 1.27" rpy="1.5708 0 1.5708"/>
+      <geometry>
+        <mesh filename="package://pf400_description/meshes/pipette.STL" scale="0.001 0.001 0.001"/>
+      </geometry>
+      <material name="black"/>
+    </visual>
+    <collision>
+      <geometry>
+        <mesh filename="package://pf400_description/meshes/pipette.STL" scale="0.001 0.001 0.001"/>
+      </geometry>
+      <origin xyz="0.79 0.76 1.27" rpy="1.5708 0 1.5708"/>
+    </collision>
+  </link>
+  <link name="${prefix}OT2_8_channel_pipette_alpha">
+    <visual>
+      <origin xyz="0.51 1.15 1.042" rpy="0 0 0"/>
+      <geometry>
+        <mesh filename="package://pf400_description/meshes/OT2_8ch_pipette.stl" scale="1 1 1"/>
+      </geometry>
+      <material name="black"/>
+    </visual>
+    <collision>
+      <geometry>
+        <mesh filename="package://pf400_description/meshes/OT2_8ch_pipette.stl" scale="1 1 1"/>
+      </geometry>
+      <origin xyz="0.51 1.15 1.042" rpy="0 0 0"/>
+    </collision>
+  </link>
+  <link name="${prefix}OT2_betha">
+    <visual>
+      <origin xyz="0.36 0.94 1.042" rpy="0 0 0"/>
+      <geometry>
+        <mesh filename="package://pf400_description/meshes/OT2_base.stl" scale="1 1 1"/>
+      </geometry>
+      <material name="aluminum"/>
+    </visual>
+    <collision>
+      <geometry>
+        <mesh filename="package://pf400_description/meshes/OT2_base.stl" scale="1 1 1"/>
+      </geometry>
+      <origin xyz="0.36 0.94 1.042" rpy="0 0 0"/>
+    </collision>
+  </link>
+  <link name="${prefix}OT2_pipette_rail_betha">
+    <visual>
+      <origin xyz="0.36 1.15 1.042" rpy="0 0 0"/>
+      <geometry>
+        <mesh filename="package://pf400_description/meshes/OT2_rail.stl" scale="1 1 1"/>
+      </geometry>
+      <material name="aluminum"/>
+    </visual>
+    <collision>
+      <geometry>
+        <mesh filename="package://pf400_description/meshes/OT2_rail.stl" scale="1 1 1"/>
+      </geometry>
+      <origin xyz="0.36 1.15 1.042" rpy="0 0 0"/>
+    </collision>
+  </link>
+  <link name="${prefix}OT2_pipette_base_betha">
+    <visual>
+      <origin xyz="0.51 1.15 1.042" rpy="0 0 0"/>
+      <geometry>
+        <mesh filename="package://pf400_description/meshes/OT2_pipette_base.stl" scale="1 1 1"/>
+      </geometry>
+      <material name="aluminum"/>
+    </visual>
+    <collision>
+      <geometry>
+        <mesh filename="package://pf400_description/meshes/OT2_pipette_base.stl" scale="1 1 1"/>
+      </geometry>
+      <origin xyz="0.51 1.15 1.042" rpy="0 0 0"/>
+    </collision>
+  </link>
+  <link name="${prefix}OT2_single_pipette_betha">
+    <visual>
+      <origin xyz="0.79 0.76 1.27" rpy="1.5708 0 1.5708"/>
+      <geometry>
+        <mesh filename="package://pf400_description/meshes/pipette.STL" scale="0.001 0.001 0.001"/>
+      </geometry>
+      <material name="black"/>
+    </visual>
+    <collision>
+      <geometry>
+        <mesh filename="package://pf400_description/meshes/pipette.STL" scale="0.001 0.001 0.001"/>
+      </geometry>
+      <origin xyz="0.79 0.76 1.27" rpy="1.5708 0 1.5708"/>
+    </collision>
+  </link>
+  <link name="${prefix}OT2_8_channel_pipette_betha">
+    <visual>
+      <origin xyz="0.51 1.15 1.042" rpy="0 0 0"/>
+      <geometry>
+        <mesh filename="package://pf400_description/meshes/OT2_8ch_pipette.stl" scale="1 1 1"/>
+      </geometry>
+      <material name="black"/>
+    </visual>
+    <collision>
+      <geometry>
+        <mesh filename="package://pf400_description/meshes/OT2_8ch_pipette.stl" scale="1 1 1"/>
+      </geometry>
+      <origin xyz="0.51 1.15 1.042" rpy="0 0 0"/>
+    </collision>
   </link>
   <!-- Joints -->
-  <joint name="OT2_1_Pipette_Joint1" type="fixed">
-    <parent link="${prefix}OT2"/>
-    <child link="${prefix}OT2_pipette_rail"/>
+  <joint name="OT2_1_Pipette_Joint1_alpha" type="fixed">
+    <parent link="${prefix}OT2_alpha"/>
+    <child link="${prefix}OT2_pipette_rail_alpha"/>
     <axis xyz="0 -1 0"/>
     <origin xyz="0 0 0" rpy="0 0 0"/>
     <limit effort="1000.0" lower="0" upper="0.3" velocity="0.5"/>
   </joint>
-  <joint name="OT2_1_Pipette_Joint2" type="fixed">
-    <parent link="${prefix}OT2_pipette_rail"/>
-    <child link="${prefix}OT2_pipette_base"/>
+  <joint name="OT2_1_Pipette_Joint2_alpha" type="fixed">
+    <parent link="${prefix}OT2_pipette_rail_alpha"/>
+    <child link="${prefix}OT2_pipette_base_alpha"/>
     <axis xyz="-1 0 0"/>
     <origin xyz="0 0 0" rpy="0 0 0"/>
     <limit effort="1000.0" lower="0" upper="0.3" velocity="0.5"/>
   </joint>
-  <joint name="OT2_1_Single_Pipette" type="fixed">
-    <parent link="${prefix}OT2_pipette_base"/>
-    <child link="${prefix}OT2_single_pipette"/>
-    <axis xyz="0 0 -1"/>
-    <origin xyz="0 0 0" rpy="0 0 0"/>
-    <limit effort="1000.0" lower="0" upper="0.18" velocity="0.5"/>
-  </joint>
-  <joint name="OT2_1_8_Channel_Pipette" type="fixed">
-    <parent link="${prefix}OT2_pipette_base"/>
-    <child link="${prefix}OT2_8_channel_pipette"/>
+  <joint name="OT2_1_Single_Pipette_alpha" type="fixed">
+    <parent link="${prefix}OT2_pipette_base_alpha"/>
+    <child link="${prefix}OT2_single_pipette_alpha"/>
+    <axis xyz="0 0 -1"/>
+    <origin xyz="0 0 0" rpy="0 0 0"/>
+    <limit effort="1000.0" lower="0" upper="0.18" velocity="0.5"/>
+  </joint>
+  <joint name="OT2_1_8_Channel_Pipette_alpha" type="fixed">
+    <parent link="${prefix}OT2_pipette_base_alpha"/>
+    <child link="${prefix}OT2_8_channel_pipette_alpha"/>
+    <axis xyz="0 0 -1"/>
+    <origin xyz="0 0 0" rpy="0 0 0"/>
+    <limit effort="1000.0" lower="0" upper="0.18" velocity="0.5"/>
+  </joint>
+  <joint name="OT2_1_Pipette_Joint1_betha" type="fixed">
+    <parent link="${prefix}OT2_betha"/>
+    <child link="${prefix}OT2_pipette_rail_betha"/>
+    <axis xyz="0 -1 0"/>
+    <origin xyz="0 0 0" rpy="0 0 0"/>
+    <limit effort="1000.0" lower="0" upper="0.3" velocity="0.5"/>
+  </joint>
+  <joint name="OT2_1_Pipette_Joint2_betha" type="fixed">
+    <parent link="${prefix}OT2_pipette_rail_betha"/>
+    <child link="${prefix}OT2_pipette_base_betha"/>
+    <axis xyz="-1 0 0"/>
+    <origin xyz="0 0 0" rpy="0 0 0"/>
+    <limit effort="1000.0" lower="0" upper="0.3" velocity="0.5"/>
+  </joint>
+  <joint name="OT2_1_Single_Pipette_betha" type="fixed">
+    <parent link="${prefix}OT2_pipette_base_betha"/>
+    <child link="${prefix}OT2_single_pipette_betha"/>
+    <axis xyz="0 0 -1"/>
+    <origin xyz="0 0 0" rpy="0 0 0"/>
+    <limit effort="1000.0" lower="0" upper="0.18" velocity="0.5"/>
+  </joint>
+  <joint name="OT2_1_8_Channel_Pipette_betha" type="fixed">
+    <parent link="${prefix}OT2_pipette_base_betha"/>
+    <child link="${prefix}OT2_8_channel_pipette_betha"/>
     <axis xyz="0 0 -1"/>
     <origin xyz="0 0 0" rpy="0 0 0"/>
