Commit message: Fixed the joint pose

File: pf400_description/urdf/hidex.urdf.xacro (robot description, xacro)
@@ -5,5 +5,5 @@
     <link name="${prefix}hidex_body">
     <visual>
-      <origin xyz="0 0 0" rpy="1.5708 0 0"/>
+      <origin xyz="0 0 0" rpy="0 0 0"/>
       <geometry>
         <mesh filename="package://pf400_description/meshes/hidex_body.STL" scale="0.001 0.001 0.001"/>
@@ -15,10 +15,10 @@
         <mesh filename="package://pf400_description/meshes/hidex_body.STL" scale="0.001 0.001 0.001"/>
       </geometry>
-      <origin xyz="0 0 0" rpy="1.5708 0 0"/>
+      <origin xyz="0 0 0" rpy="0 0 0"/>
     </collision>
   </link>
   <link name="${prefix}hidex_plate">
     <visual>
-      <origin xyz="0 0 0" rpy="0 1.5708 0"/>
+      <origin xyz="0 0 0" rpy="0 0 0"/>
       <geometry>
         <mesh filename="package://pf400_description/meshes/hidex_plate.STL" scale="0.001 0.001 0.001"/>
@@ -30,5 +30,5 @@
         <mesh filename="package://pf400_description/meshes/hidex_plate.STL" scale="0.001 0.001 0.001"/>
       </geometry>
-      <origin xyz="0 0 0" rpy="0 1.5708 0"/>
+      <origin xyz="0 0 0" rpy="0 0 0"/>
     </collision>
   </link>
@@ -38,5 +38,5 @@
     <child link="${prefix}hidex_plate"/>
     <axis xyz="0 0 1"/>
-    <origin xyz="0.25 -0.18 0.083" rpy="1.5708 0 0"/>
+    <origin xyz="0.055 -0.09 0.065" rpy="0 0 0"/>
     <limit effort="1000.0" lower="0" upper="0.3" velocity="0.5"/>
   </joint>
