Commit message: Xacro files are not working yet

File: pf400_description/urdf/pcr_workcell.urdf.xacro (robot description, xacro)
@@ -228,145 +228,11 @@
     </visual>
   </link>
-  <link name="rail_base">
-    <visual>
-      <origin xyz="0.125 -0.0198 1.015" rpy="0 0 1.5708"/>
-      <geometry>
-        <mesh filename="package://pf400_description/meshes/rail_base.STL" scale="1 1 1"/>
-      </geometry>
-      <material name="white"/>
-    </visual>
-  </link>
-  <link name="rail">
-    <visual>
-      <origin xyz="0.1309 -0.0198 1.047" rpy="1.5708 0 1.5708"/>
-      <geometry>
-        <mesh filename="package://pf400_description/meshes/rail.STL" scale="1 1 1"/>
-      </geometry>
-      <material name="white"/>
-    </visual>
-  </link>
-  <link name="z_column">
-    <visual>
-      <origin xyz="0 0 1.089" rpy="0 0 0"/>
-      <geometry>
-        <mesh filename="package://pf400_description/meshes/PF400_Z_Column.STL" scale="0.001 0.001 0.00132"/>
-      </geometry>
-      <material name="white"/>
-    </visual>
-  </link>
-  <link name="z_carriage">
-    <visual>
-      <origin xyz="0 0 1.089" rpy="0 0 0"/>
-      <geometry>
-        <mesh filename="package://pf400_description/meshes/PF400_Z_Carriage.STL" scale="0.001 0.001 0.001"/>
-      </geometry>
-      <material name="white"/>
-    </visual>
-  </link>
-  <link name="inner_link">
-    <visual>
-      <origin xyz="0 0 1.089" rpy="0 0 0"/>
-      <geometry>
-        <mesh filename="package://pf400_description/meshes/PF400_Inner_Link.STL" scale="0.001 0.001 0.001"/>
-      </geometry>
-      <material name="white"/>
-    </visual>
-  </link>
-  <link name="outer_link">
-    <visual>
-      <origin xyz="0 0 1.089" rpy="0 0 0"/>
-      <geometry>
-        <mesh filename="package://pf400_description/meshes/PF400_Outer_Link.STL" scale="0.001 0.001 0.001"/>
-      </geometry>
-      <material name="white"/>
-    </visual>
-  </link>
-  <link name="hand">
-    <visual>
-      <origin xyz="0 0 1.089" rpy="0 0 0"/>
-      <geometry>
-        <mesh filename="package://pf400_description/meshes/PF400_Hand.STL" scale="0.001 0.001 0.001"/>
-      </geometry>
-      <material name="white"/>
-    </visual>
-  </link>
-  <link name="left_finger">
-    <visual>
-      <origin xyz="-0.02 -0.053 1.0685" rpy="0 0 0"/>
-      <geometry>
-        <mesh filename="package://pf400_description/meshes/pf400_left_finger.STL" scale="0.001 0.001 0.001"/>
-      </geometry>
-      <material name="aluminum"/>
-    </visual>
-  </link>
-  <link name="right_finger">
-    <visual>
-      <origin xyz="-0.021 -0.028 1.12" rpy="-1.5708 0 0"/>
-      <geometry>
-        <mesh filename="package://pf400_description/meshes/pf400_right_finger.STL" scale="0.001 0.001 0.001"/>
-      </geometry>
-      <material name="aluminum"/>
-    </visual>
-  </link>
+  <!-- PF400 -->
+  <xacro:include filename="$(find pf400_description)/urdf/PF400.urdf.xacro" />
+  <xacro:pf400 prefix="${prefix}pf400/"/>
   <!-- Joints -->
-  <joint name="J1" type="prismatic">
-    <parent link="z_column"/>
-    <child link="z_carriage"/>
-    <axis xyz="0 0 1"/>
-    <origin xyz="0.03005 -0.0198 0.17535" rpy="0 0 0"/>
-    <limit effort="1000.0" lower="0.002" upper="1.160" velocity="0.5"/>  </joint>
-  <joint name="J2" type="revolute">
-    <parent link="z_carriage"/>
-    <child link="inner_link"/>
-    <axis xyz="0 0 1"/>
-    <origin xyz="0.173001 0.020 0.0235" rpy="0 0 0"/>
-    <limit effort="1000.0" lower="-1.62316" upper="1.62316" velocity="0.5"/>
-  </joint>
-  <joint name="J3" type="revolute">
-    <parent link="inner_link"/>
-    <child link="outer_link"/>
-    <axis xyz="0 0 1"/>
-    <origin xyz="0.302 0 -0.072285" rpy="0 0 0"/>
-    <limit effort="1000.0" lower="0.175" upper="6.1" velocity="0.5"/>
-  </joint>
-  <joint name="J4" type="revolute">
-    <parent link="outer_link"/>
-    <child link="hand"/>
-    <axis xyz="0 0 1"/>
-    <origin xyz="0.289 0 -0.032942" rpy="0 0 0"/>
-    <limit effort="1000.0" lower="-16.7552" upper="16.7552" velocity="0.5"/>
-  </joint>
-  <joint name="J5" type="prismatic">
-    <parent link="hand"/>
-    <child link="left_finger"/>
-    <axis xyz="0 1 0"/>
-    <origin xyz="0.078573 0 -0.04269" rpy="0 0 0"/>
-    <limit effort="1000.0" lower="0.04" upper="0.0675" velocity="0.5"/>
-  </joint>
-  <joint name="J5_mirror" type="prismatic">
-    <parent link="hand"/>
-    <child link="right_finger"/>
-    <axis xyz="0 -1 0"/>
-    <origin xyz="0.078573 0 -0.04269" rpy="0 0 0"/>
-    <limit effort="1000.0" lower="0.04" upper="0.0675" velocity="0.5"/>
-    <mimic joint="J5" multiplier="1"/>
-  </joint>
-  <joint name="J6" type="prismatic">
-    <parent link="rail_base"/>
-    <child link="rail"/>
-    <axis xyz="1 0 0"/>
-    <origin xyz="0 0 0" rpy="0 0 0"/>
-    <limit effort="1000.0" lower="-1" upper="1" velocity="0.5"/>
-  </joint>
-  <joint name="rail_link" type="fixed">
-    <parent link="rail"/>
-    <child link="z_column"/>
-    <axis xyz="0 1 0"/>
-    <origin xyz="0.03005 -0.0198 0.05" rpy="0 0 0"/>
-    <limit effort="1000.0" lower="0" upper="0" velocity="0.5"/>
-  </joint>
   <joint name="module_table" type="fixed">
     <parent link="pf400_module"/>
-    <child link="rail_base"/>
+    <child link="${prefix}pf400/rail_base"/>
     <axis xyz="0 0 1"/>
     <origin xyz="0 0 0" rpy="0 0 0"/>

Commit message: Fixing description imports

File: pf400_description/urdf/pcr_workcell.urdf.xacro (robot description, xacro)
@@ -35,11 +35,11 @@
     <parent link="module_carts/pf400_cart"/>
     <child link="pf400/rail_base"/>
-    <axis xyz="0 0 1"/>
-    <origin xyz="0 0 0" rpy="0 0 0"/>
+    <axis xyz="0 0 0"/>
+    <origin xyz="0.125 -0.0198 1.015" rpy="0 0 0"/>
     <limit effort="1000.0" lower="0" upper="0" velocity="0.5"/>
   </joint>
   <joint name="Thermocycler_Base" type="fixed">
     <parent link="module_carts/cart_4"/>
-    <child link="thermocycler/Thermocycler_Base"/>
+    <child link="thermocycler/thermocycler_base"/>
     <axis xyz="0 0 1"/>
     <origin xyz="-0.2 0.2 0" rpy="0 0 0"/>

Commit message: RPL commit

File: pf400_description/urdf/pcr_workcell.urdf.xacro (robot description, xacro)
@@ -36,5 +36,5 @@
     <child link="pf400/rail_base"/>
     <axis xyz="0 0 0"/>
-    <origin xyz="0.125 -0.0198 1.015" rpy="0 0 0"/>
+    <origin xyz="0 -0.0198 1.015" rpy="0 0 0"/>
     <limit effort="1000.0" lower="0" upper="0" velocity="0.5"/>
   </joint>

Commit message: Fixing pf400 location

File: pf400_description/urdf/pcr_workcell.urdf.xacro (robot description, xacro)
@@ -36,5 +36,5 @@
     <child link="pf400/rail_base"/>
     <axis xyz="0 0 0"/>
-    <origin xyz="0 -0.0198 1.015" rpy="0 0 0"/>
+    <origin xyz="-0.14 -0.0198 1.015" rpy="0 0 0"/>
     <limit effort="1000.0" lower="0" upper="0" velocity="0.5"/>
   </joint>

Commit message: Fixing pf400 hight

File: pf400_description/urdf/pcr_workcell.urdf.xacro (robot description, xacro)
@@ -36,5 +36,5 @@
     <child link="pf400/rail_base"/>
     <axis xyz="0 0 0"/>
-    <origin xyz="-0.14 -0.0198 1.015" rpy="0 0 0"/>
+    <origin xyz="-0.14 -0.0198 0.83" rpy="0 0 0"/>
     <limit effort="1000.0" lower="0" upper="0" velocity="0.5"/>
   </joint>

Commit message: Fixing pf400 hight

File: pf400_description/urdf/pcr_workcell.urdf.xacro (robot description, xacro)
@@ -36,5 +36,5 @@
     <child link="pf400/rail_base"/>
     <axis xyz="0 0 0"/>
-    <origin xyz="-0.14 -0.0198 0.83" rpy="0 0 0"/>
+    <origin xyz="-0.14 -0.0198 0.835" rpy="0 0 0"/>
     <limit effort="1000.0" lower="0" upper="0" velocity="0.5"/>
   </joint>

Commit message: Fixing all the module locations

File: pf400_description/urdf/pcr_workcell.urdf.xacro (robot description, xacro)
@@ -24,5 +24,5 @@
   <link name="OT2_2">
     <visual>
-      <origin xyz="0.975 -1.02 1.042" rpy="1.5708 0 3.1416"/>
+      <origin xyz="0 0 0" rpy="1.5708 0 3.1416"/>
       <geometry>
         <mesh filename="package://pf400_description/meshes/OT_2_without_pipette.STL" scale="0.001 0.001 0.001"/>
@@ -40,36 +40,43 @@
   </joint>
   <joint name="Thermocycler_Base" type="fixed">
-    <parent link="module_carts/cart_4"/>
+    <parent link="module_carts/cart_2"/>
     <child link="thermocycler/thermocycler_base"/>
     <axis xyz="0 0 1"/>
-    <origin xyz="-0.2 0.2 0" rpy="0 0 0"/>
+    <origin xyz="0.2 -0.65 0" rpy="0 0 0"/>
+    <limit effort="1000.0" lower="0" upper="0" velocity="0.5"/>
+  </joint>
+  <joint name="Thermocycler_Base2" type="fixed">
+    <parent link="module_carts/cart_2"/>
+    <child link="thermocycler/thermocycler_base2"/>
+    <axis xyz="0 0 1"/>
+    <origin xyz="-0.1 -0.65 0" rpy="0 0 0"/>
     <limit effort="1000.0" lower="0" upper="0" velocity="0.5"/>
   </joint>
   <joint name="Peeler_Base" type="fixed">
-    <parent link="module_carts/cart_5"/>
+    <parent link="module_carts/cart_6"/>
     <child link="peeler/peeler_base"/>
     <axis xyz="0 0 0"/>
-    <origin xyz="1.15 -0.37 1.042" rpy="0 0 0"/>
+    <origin xyz="-0.17 0.19 1.042" rpy="0 0 0"/>
     <limit effort="1000.0" lower="0" upper="0" velocity="0.5"/>
   </joint>
   <joint name="Sealer_Base" type="fixed">
-    <parent link="module_carts/cart_5"/>
+    <parent link="module_carts/cart_6"/>
     <child link="sealer/sealer_base"/>
     <axis xyz="0 0 1"/>
-    <origin xyz="1.55 -1.05 1.042" rpy="0 0 0"/>
+    <origin xyz="0.23 -0.51 1.042" rpy="0 0 0"/>
     <limit effort="1000.0" lower="0" upper="0" velocity="0.5"/>
   </joint>
   <joint name="OT2" type="fixed">
-    <parent link="module_carts/cart_2"/>
+    <parent link="module_carts/cart_8"/>
     <child link="ot2/OT2"/>
     <axis xyz="0 0 1"/>
-    <origin xyz="0 0 0" rpy="0 0 0"/>
+    <origin xyz="0.825 0.47 0" rpy="0 0 3.1416"/>
     <limit effort="1000.0" lower="0" upper="0" velocity="0.5"/>
   </joint>
   <joint name="OT2_2" type="fixed">
-    <parent link="ot2/OT2"/>
+    <parent link="module_carts/cart_7"/>
     <child link="OT2_2"/>
     <axis xyz="0 0 1"/>
-    <origin xyz="0 0 0" rpy="0 0 0"/>
+    <origin xyz="0.465 -0.47 1.04" rpy="0 0 0"/>
     <limit effort="1000.0" lower="0" upper="0" velocity="0.5"/>
   </joint>

Commit message: Adding OT2_alpha and OT2_betha

File: pf400_description/urdf/pcr_workcell.urdf.xacro (robot description, xacro)
@@ -21,15 +21,5 @@
   <xacro:include filename="$(find pf400_description)/urdf/module_carts.urdf.xacro" />
   <xacro:Module_Carts prefix="module_carts/"/>
-  <!-- Links -->
-  <link name="OT2_2">
-    <visual>
-      <origin xyz="0 0 0" rpy="1.5708 0 3.1416"/>
-      <geometry>
-        <mesh filename="package://pf400_description/meshes/OT_2_without_pipette.STL" scale="0.001 0.001 0.001"/>
-      </geometry>
-      <material name="aluminum"/>
-    </visual>
-  </link>
-  <!-- Joints -->
+  <!-- Wrokcell Setup -->
   <joint name="pf400_module" type="fixed">
     <parent link="module_carts/pf400_cart"/>
@@ -42,5 +32,5 @@
     <parent link="module_carts/cart_2"/>
     <child link="thermocycler/thermocycler_base"/>
-    <axis xyz="0 0 1"/>
+    <axis xyz="0 0 0"/>
     <origin xyz="0.2 -0.65 0" rpy="0 0 0"/>
     <limit effort="1000.0" lower="0" upper="0" velocity="0.5"/>
@@ -49,5 +39,5 @@
     <parent link="module_carts/cart_2"/>
     <child link="thermocycler/thermocycler_base2"/>
-    <axis xyz="0 0 1"/>
+    <axis xyz="0 0 0"/>
     <origin xyz="-0.1 -0.65 0" rpy="0 0 0"/>
     <limit effort="1000.0" lower="0" upper="0" velocity="0.5"/>
@@ -63,20 +53,20 @@
     <parent link="module_carts/cart_6"/>
     <child link="sealer/sealer_base"/>
-    <axis xyz="0 0 1"/>
+    <axis xyz="0 0 0"/>
     <origin xyz="0.23 -0.51 1.042" rpy="0 0 0"/>
     <limit effort="1000.0" lower="0" upper="0" velocity="0.5"/>
   </joint>
-  <joint name="OT2" type="fixed">
+  <joint name="OT2_alpha" type="fixed">
     <parent link="module_carts/cart_8"/>
-    <child link="ot2/OT2"/>
-    <axis xyz="0 0 1"/>
+    <child link="ot2/OT2_alpha"/>
+    <axis xyz="0 0 0"/>
     <origin xyz="0.825 0.47 0" rpy="0 0 3.1416"/>
     <limit effort="1000.0" lower="0" upper="0" velocity="0.5"/>
   </joint>
-  <joint name="OT2_2" type="fixed">
+  <joint name="OT2_betha" type="fixed">
     <parent link="module_carts/cart_7"/>
-    <child link="OT2_2"/>
-    <axis xyz="0 0 1"/>
-    <origin xyz="0.465 -0.47 1.04" rpy="0 0 0"/>
+    <child link="ot2/OT2_betha"/>
+    <axis xyz="0 0 0"/>
+    <origin xyz="0.825 0.47 0" rpy="0 0 3.1416"/>
     <limit effort="1000.0" lower="0" upper="0" velocity="0.5"/>
   </joint>

Commit message: Adding Hidex into pcr description

File: pf400_description/urdf/pcr_workcell.urdf.xacro (robot description, xacro)
@@ -18,4 +18,7 @@
   <xacro:include filename="$(find pf400_description)/urdf/thermocycler.urdf.xacro" />
   <xacro:Thermocycler prefix="thermocycler/"/>
+  <!-- Hidex -->
+  <xacro:include filename="$(find pf400_description)/urdf/hidex.urdf.xacro" />
+  <xacro:Hidex prefix="hidex/"/>
   <!-- Module Carts -->
   <xacro:include filename="$(find pf400_description)/urdf/module_carts.urdf.xacro" />
@@ -57,4 +60,11 @@
     <limit effort="1000.0" lower="0" upper="0" velocity="0.5"/>
   </joint>
+  <joint name="Hidex_Base" type="fixed">
+    <parent link="module_carts/cart_3"/>
+    <child link="hidex/hidex_body"/>
+    <axis xyz="0 0 0"/>
+    <origin xyz="0.23 -0.51 1.042" rpy="0 0 0"/>
+    <limit effort="1000.0" lower="0" upper="0" velocity="0.5"/>
+  </joint>
   <joint name="OT2_alpha" type="fixed">
     <parent link="module_carts/cart_8"/>

Commit message: Added Hidex description

File: pf400_description/urdf/pcr_workcell.urdf.xacro (robot description, xacro)
@@ -64,5 +64,5 @@
     <child link="hidex/hidex_body"/>
     <axis xyz="0 0 0"/>
-    <origin xyz="0.23 -0.51 1.042" rpy="0 0 0"/>
+    <origin xyz="0.2 -0.45 1.042" rpy="0 0 0"/>
     <limit effort="1000.0" lower="0" upper="0" velocity="0.5"/>
   </joint>
