Commit message: pf400 xacro created

File: pf400_description/urdf/PF400.urdf.xacro (robot description, xacro)
@@ -10,15 +10,15 @@
   <!-- PF400 -->
   <xacro:include filename="$(find pf400_description)/urdf/test.urdf.xacro" />
-  <xacro:pf400 prefix="${prefix}pf400/"/>
+  <xacro:pf400 prefix="pf400/"/>
   <!-- Joints -->
   <joint name="J1" type="prismatic">
-    <parent link="${prefix}pf400/z_column"/>
-    <child link="${prefix}pf400/z_carriage"/>
+    <parent link="pf400/z_column"/>
+    <child link="pf400/z_carriage"/>
     <axis xyz="0 0 1"/>
     <origin xyz="0.03005 -0.0198 0.17535" rpy="0 0 0"/>
     <limit effort="1000.0" lower="0.002" upper="1.160" velocity="0.5"/>  </joint>
   <joint name="J2" type="revolute">
-    <parent link="${prefix}pf400/z_carriage"/>
-    <child link="${prefix}pf400/inner_link"/>
+    <parent link="pf400/z_carriage"/>
+    <child link="pf400/inner_link"/>
     <axis xyz="0 0 1"/>
     <origin xyz="0.173001 0.020 0.0235" rpy="0 0 0"/>
@@ -26,6 +26,6 @@
   </joint>
   <joint name="J3" type="revolute">
-    <parent link="${prefix}pf400/inner_link"/>
-    <child link="${prefix}pf400/outer_link"/>
+    <parent link="pf400/inner_link"/>
+    <child link="pf400/outer_link"/>
     <axis xyz="0 0 1"/>
     <origin xyz="0.302 0 -0.072285" rpy="0 0 0"/>
@@ -33,6 +33,6 @@
   </joint>
   <joint name="J4" type="revolute">
-    <parent link="${prefix}pf400/outer_link"/>
-    <child link="${prefix}pf400/hand"/>
+    <parent link="pf400/outer_link"/>
+    <child link="pf400/hand"/>
     <axis xyz="0 0 1"/>
     <origin xyz="0.289 0 -0.032942" rpy="0 0 0"/>
@@ -40,6 +40,6 @@
   </joint>
   <joint name="J5" type="prismatic">
-    <parent link="${prefix}pf400/hand"/>
-    <child link="${prefix}pf400/left_finger"/>
+    <parent link="pf400/hand"/>
+    <child link="pf400/left_finger"/>
     <axis xyz="0 1 0"/>
     <origin xyz="0.078573 0 -0.04269" rpy="0 0 0"/>
@@ -47,6 +47,6 @@
   </joint>
   <joint name="J5_mirror" type="prismatic">
-    <parent link="${prefix}pf400/hand"/>
-    <child link="${prefix}pf400/right_finger"/>
+    <parent link="pf400/hand"/>
+    <child link="pf400/right_finger"/>
     <axis xyz="0 -1 0"/>
     <origin xyz="0.078573 0 -0.04269" rpy="0 0 0"/>
@@ -55,6 +55,6 @@
   </joint>
   <joint name="J6" type="prismatic">
-    <parent link="${prefix}pf400/rail_base"/>
-    <child link="${prefix}pf400/rail"/>
+    <parent link="pf400/rail_base"/>
+    <child link="pf400/rail"/>
     <axis xyz="1 0 0"/>
     <origin xyz="0 0 0" rpy="0 0 0"/>
@@ -62,6 +62,6 @@
   </joint>
   <joint name="rail_link" type="fixed">
-    <parent link="${prefix}pf400/rail"/>
-    <child link="${prefix}pf400/z_column"/>
+    <parent link="pf400/rail"/>
+    <child link="pf400/z_column"/>
     <axis xyz="0 1 0"/>
     <origin xyz="0.03005 -0.0198 0.05" rpy="0 0 0"/>

File: pf400_description/urdf/test.urdf.xacro (robot description, xacro)
@@ -3,5 +3,5 @@
   <!-- Links -->
   <xacro:macro name="pf400" params = "prefix">
-  <link name="${prefix}pf400/rail_base">
+  <link name="${prefix}rail_base">
     <visual>
       <origin xyz="0.125 -0.0198 0" rpy="0 0 1.5708"/>
@@ -12,5 +12,5 @@
     </visual>
   </link>
-  <link name="${prefix}pf400/rail">
+  <link name="${prefix}rail">
     <visual>
       <origin xyz="0.1309 -0.0198 0.0320" rpy="1.5708 0 1.5708"/>
@@ -21,5 +21,5 @@
     </visual>
   </link>
-  <link name="${prefix}pf400/z_column">
+  <link name="${prefix}z_column">
     <visual>
       <origin xyz="0 0 0.074" rpy="0 0 0"/>
@@ -30,5 +30,5 @@
     </visual>
   </link>
-  <link name="${prefix}pf400/z_carriage">
+  <link name="${prefix}z_carriage">
     <visual>
       <origin xyz="0 0 0.074" rpy="0 0 0"/>
@@ -39,5 +39,5 @@
     </visual>
   </link>
-  <link name="${prefix}pf400/inner_link">
+  <link name="${prefix}inner_link">
     <visual>
       <origin xyz="0 0 0.074" rpy="0 0 0"/>
@@ -48,5 +48,5 @@
     </visual>
   </link>
-  <link name="${prefix}pf400/outer_link">
+  <link name="${prefix}outer_link">
     <visual>
       <origin xyz="0 0 0.074" rpy="0 0 0"/>
@@ -57,5 +57,5 @@
     </visual>
   </link>
-  <link name="${prefix}pf400/hand">
+  <link name="${prefix}hand">
     <visual>
       <origin xyz="0 0 0.074" rpy="0 0 0"/>
@@ -66,5 +66,5 @@
     </visual>
   </link>
-  <link name="${prefix}pf400/left_finger">
+  <link name="${prefix}left_finger">
     <visual>
       <origin xyz="-0.02 -0.053 0.053" rpy="0 0 0"/>
@@ -75,5 +75,5 @@
     </visual>
   </link>
-  <link name="${prefix}pf400/right_finger">
+  <link name="${prefix}right_finger">
     <visual>
       <origin xyz="-0.021 -0.028 0.105" rpy="-1.5708 0 0"/>

Commit message: Working individual robot xacro files

File: pf400_description/urdf/PF400.urdf.xacro (robot description, xacro)
@@ -1,24 +1,97 @@
 <?xml version="1.0"?>
 <robot name="PF400_Robot" xmlns:xacro="http://www.ros.org/wiki/xacro">
-  <!-- Materials -->
-  <material name="white">
-    <color rgba="1 1 1 1"/>
-  </material>
-  <material name="aluminum">
-    <color rgba="0.6 0.6 0.6 1"/>
-  </material>
-  <!-- PF400 -->
-  <xacro:include filename="$(find pf400_description)/urdf/test.urdf.xacro" />
-  <xacro:pf400 prefix="pf400/"/>
+  <!-- Links -->
+  <xacro:macro name="pf400" params = "prefix">
+  <link name="${prefix}rail_base">
+    <visual>
+      <origin xyz="0.125 -0.0198 0" rpy="0 0 1.5708"/>
+      <geometry>
+        <mesh filename="package://pf400_description/meshes/rail_base.STL" scale="1 1 1"/>
+      </geometry>
+      <material name="white"/>
+    </visual>
+  </link>
+  <link name="${prefix}rail">
+    <visual>
+      <origin xyz="0.1309 -0.0198 0.0320" rpy="1.5708 0 1.5708"/>
+      <geometry>
+        <mesh filename="package://pf400_description/meshes/rail.STL" scale="1 1 1"/>
+      </geometry>
+      <material name="white"/>
+    </visual>
+  </link>
+  <link name="${prefix}z_column">
+    <visual>
+      <origin xyz="0 0 0.074" rpy="0 0 0"/>
+      <geometry>
+        <mesh filename="package://pf400_description/meshes/PF400_Z_Column.STL" scale="0.001 0.001 0.00132"/>
+      </geometry>
+      <material name="white"/>
+    </visual>
+  </link>
+  <link name="${prefix}z_carriage">
+    <visual>
+      <origin xyz="0 0 0.074" rpy="0 0 0"/>
+      <geometry>
+        <mesh filename="package://pf400_description/meshes/PF400_Z_Carriage.STL" scale="0.001 0.001 0.001"/>
+      </geometry>
+      <material name="white"/>
+    </visual>
+  </link>
+  <link name="${prefix}inner_link">
+    <visual>
+      <origin xyz="0 0 0.074" rpy="0 0 0"/>
+      <geometry>
+        <mesh filename="package://pf400_description/meshes/PF400_Inner_Link.STL" scale="0.001 0.001 0.001"/>
+      </geometry>
+      <material name="white"/>
+    </visual>
+  </link>
+  <link name="${prefix}outer_link">
+    <visual>
+      <origin xyz="0 0 0.074" rpy="0 0 0"/>
+      <geometry>
+        <mesh filename="package://pf400_description/meshes/PF400_Outer_Link.STL" scale="0.001 0.001 0.001"/>
+      </geometry>
+      <material name="white"/>
+    </visual>
+  </link>
+  <link name="${prefix}hand">
+    <visual>
+      <origin xyz="0 0 0.074" rpy="0 0 0"/>
+      <geometry>
+        <mesh filename="package://pf400_description/meshes/PF400_Hand.STL" scale="0.001 0.001 0.001"/>
+      </geometry>
+      <material name="white"/>
+    </visual>
+  </link>
+  <link name="${prefix}left_finger">
+    <visual>
+      <origin xyz="-0.02 -0.053 0.053" rpy="0 0 0"/>
+      <geometry>
+        <mesh filename="package://pf400_description/meshes/pf400_left_finger.STL" scale="0.001 0.001 0.001"/>
+      </geometry>
+      <material name="aluminum"/>
+    </visual>
+  </link>
+  <link name="${prefix}right_finger">
+    <visual>
+      <origin xyz="-0.021 -0.028 0.105" rpy="-1.5708 0 0"/>
+      <geometry>
+        <mesh filename="package://pf400_description/meshes/pf400_right_finger.STL" scale="0.001 0.001 0.001"/>
+      </geometry>
+      <material name="aluminum"/>
+    </visual>
+  </link>
   <!-- Joints -->
   <joint name="J1" type="prismatic">
-    <parent link="pf400/z_column"/>
-    <child link="pf400/z_carriage"/>
+    <parent link="${prefix}z_column"/>
+    <child link="${prefix}z_carriage"/>
     <axis xyz="0 0 1"/>
     <origin xyz="0.03005 -0.0198 0.17535" rpy="0 0 0"/>
     <limit effort="1000.0" lower="0.002" upper="1.160" velocity="0.5"/>  </joint>
   <joint name="J2" type="revolute">
-    <parent link="pf400/z_carriage"/>
-    <child link="pf400/inner_link"/>
+    <parent link="${prefix}z_carriage"/>
+    <child link="${prefix}inner_link"/>
     <axis xyz="0 0 1"/>
     <origin xyz="0.173001 0.020 0.0235" rpy="0 0 0"/>
@@ -26,6 +99,6 @@
   </joint>
   <joint name="J3" type="revolute">
-    <parent link="pf400/inner_link"/>
-    <child link="pf400/outer_link"/>
+    <parent link="${prefix}inner_link"/>
+    <child link="${prefix}outer_link"/>
     <axis xyz="0 0 1"/>
     <origin xyz="0.302 0 -0.072285" rpy="0 0 0"/>
@@ -33,6 +106,6 @@
   </joint>
   <joint name="J4" type="revolute">
-    <parent link="pf400/outer_link"/>
-    <child link="pf400/hand"/>
+    <parent link="${prefix}outer_link"/>
+    <child link="${prefix}hand"/>
     <axis xyz="0 0 1"/>
     <origin xyz="0.289 0 -0.032942" rpy="0 0 0"/>
@@ -40,6 +113,6 @@
   </joint>
   <joint name="J5" type="prismatic">
-    <parent link="pf400/hand"/>
-    <child link="pf400/left_finger"/>
+    <parent link="${prefix}hand"/>
+    <child link="${prefix}left_finger"/>
     <axis xyz="0 1 0"/>
     <origin xyz="0.078573 0 -0.04269" rpy="0 0 0"/>
@@ -47,6 +120,6 @@
   </joint>
   <joint name="J5_mirror" type="prismatic">
-    <parent link="pf400/hand"/>
-    <child link="pf400/right_finger"/>
+    <parent link="${prefix}hand"/>
+    <child link="${prefix}right_finger"/>
     <axis xyz="0 -1 0"/>
     <origin xyz="0.078573 0 -0.04269" rpy="0 0 0"/>
@@ -55,6 +128,6 @@
   </joint>
   <joint name="J6" type="prismatic">
-    <parent link="pf400/rail_base"/>
-    <child link="pf400/rail"/>
+    <parent link="${prefix}rail_base"/>
+    <child link="${prefix}rail"/>
     <axis xyz="1 0 0"/>
     <origin xyz="0 0 0" rpy="0 0 0"/>
@@ -62,9 +135,10 @@
   </joint>
   <joint name="rail_link" type="fixed">
-    <parent link="pf400/rail"/>
-    <child link="pf400/z_column"/>
+    <parent link="${prefix}rail"/>
+    <child link="${prefix}z_column"/>
     <axis xyz="0 1 0"/>
     <origin xyz="0.03005 -0.0198 0.05" rpy="0 0 0"/>
     <limit effort="1000.0" lower="0" upper="0" velocity="0.5"/>
   </joint>
+  </xacro:macro>
 </robot>

File: pf400_description/urdf/pcr_workcell.urdf.xacro (robot description, xacro)
@@ -38,4 +38,7 @@
     <color rgba="0.6 0.6 0.6 1"/>
   </material>
+  <!-- PF400 -->
+  <xacro:include filename="$(find pf400_description)/urdf/PF400.urdf.xacro" />
+  <xacro:pf400 prefix="pf400/"/>
   <!-- Links -->
   <link name="Peeler_Base">
@@ -228,11 +231,8 @@
     </visual>
   </link>
-  <!-- PF400 -->
-  <xacro:include filename="$(find pf400_description)/urdf/PF400.urdf.xacro" />
-  <xacro:pf400 prefix="${prefix}pf400/"/>
   <!-- Joints -->
   <joint name="module_table" type="fixed">
     <parent link="pf400_module"/>
-    <child link="${prefix}pf400/rail_base"/>
+    <child link="pf400/rail_base"/>
     <axis xyz="0 0 1"/>
     <origin xyz="0 0 0" rpy="0 0 0"/>

File: pf400_description/urdf/test.urdf.xacro (robot description, xacro)
@@ -84,4 +84,60 @@
     </visual>
   </link>
+  <joint name="J1" type="prismatic">
+    <parent link="${prefix}z_column"/>
+    <child link="${prefix}z_carriage"/>
+    <axis xyz="0 0 1"/>
+    <origin xyz="0.03005 -0.0198 0.17535" rpy="0 0 0"/>
+    <limit effort="1000.0" lower="0.002" upper="1.160" velocity="0.5"/>  </joint>
+  <joint name="J2" type="revolute">
+    <parent link="${prefix}z_carriage"/>
+    <child link="${prefix}inner_link"/>
+    <axis xyz="0 0 1"/>
+    <origin xyz="0.173001 0.020 0.0235" rpy="0 0 0"/>
+    <limit effort="1000.0" lower="-1.62316" upper="1.62316" velocity="0.5"/>
+  </joint>
+  <joint name="J3" type="revolute">
+    <parent link="${prefix}inner_link"/>
+    <child link="${prefix}outer_link"/>
+    <axis xyz="0 0 1"/>
+    <origin xyz="0.302 0 -0.072285" rpy="0 0 0"/>
+    <limit effort="1000.0" lower="0.175" upper="6.1" velocity="0.5"/>
+  </joint>
+  <joint name="J4" type="revolute">
+    <parent link="${prefix}outer_link"/>
+    <child link="${prefix}hand"/>
+    <axis xyz="0 0 1"/>
+    <origin xyz="0.289 0 -0.032942" rpy="0 0 0"/>
+    <limit effort="1000.0" lower="-16.7552" upper="16.7552" velocity="0.5"/>
+  </joint>
+  <joint name="J5" type="prismatic">
+    <parent link="${prefix}hand"/>
+    <child link="${prefix}left_finger"/>
+    <axis xyz="0 1 0"/>
+    <origin xyz="0.078573 0 -0.04269" rpy="0 0 0"/>
+    <limit effort="1000.0" lower="0.067454" upper="0.070" velocity="0.5"/>
+  </joint>
+  <joint name="J5_mirror" type="prismatic">
+    <parent link="${prefix}hand"/>
+    <child link="${prefix}right_finger"/>
+    <axis xyz="0 -1 0"/>
+    <origin xyz="0.078573 0 -0.04269" rpy="0 0 0"/>
+    <limit effort="1000.0" lower="0.067454" upper="0.070" velocity="0.5"/>
+    <mimic joint="J5" multiplier="1"/>
+  </joint>
+  <joint name="J6" type="prismatic">
+    <parent link="${prefix}rail_base"/>
+    <child link="${prefix}rail"/>
+    <axis xyz="1 0 0"/>
+    <origin xyz="0 0 0" rpy="0 0 0"/>
+    <limit effort="1000.0" lower="-1" upper="1" velocity="0.5"/>
+  </joint>
+  <joint name="rail_link" type="fixed">
+    <parent link="${prefix}rail"/>
+    <child link="${prefix}z_column"/>
+    <axis xyz="0 1 0"/>
+    <origin xyz="0.03005 -0.0198 0.05" rpy="0 0 0"/>
+    <limit effort="1000.0" lower="0" upper="0" velocity="0.5"/>
+  </joint>
   </xacro:macro>
 </robot>

Commit message: Fixing robot origin

File: pf400_description/urdf/PF400.urdf.xacro (robot description, xacro)
@@ -5,5 +5,5 @@
   <link name="${prefix}rail_base">
     <visual>
-      <origin xyz="0.125 -0.0198 0" rpy="0 0 1.5708"/>
+      <origin xyz="0 0 0" rpy="0 0 1.5708"/>
       <geometry>
         <mesh filename="package://pf400_description/meshes/rail_base.STL" scale="1 1 1"/>
@@ -14,5 +14,5 @@
   <link name="${prefix}rail">
     <visual>
-      <origin xyz="0.1309 -0.0198 0.0320" rpy="1.5708 0 1.5708"/>
+      <origin xyz="0 0 0" rpy="1.5708 0 1.5708"/>
       <geometry>
         <mesh filename="package://pf400_description/meshes/rail.STL" scale="1 1 1"/>
@@ -118,5 +118,5 @@
     <axis xyz="0 1 0"/>
     <origin xyz="0.078573 0 -0.04269" rpy="0 0 0"/>
-    <limit effort="1000.0" lower="0.067454" upper="0.070" velocity="0.5"/>
+    <limit effort="1000.0" lower="0.04" upper="0.0675" velocity="0.5"/>
   </joint>
   <joint name="J5_mirror" type="prismatic">
@@ -125,5 +125,5 @@
     <axis xyz="0 -1 0"/>
     <origin xyz="0.078573 0 -0.04269" rpy="0 0 0"/>
-    <limit effort="1000.0" lower="0.067454" upper="0.070" velocity="0.5"/>
+    <limit effort="1000.0" lower="0.04" upper="0.0675" velocity="0.5"/>
     <mimic joint="J5" multiplier="1"/>
   </joint>
@@ -132,5 +132,5 @@
     <child link="${prefix}rail"/>
     <axis xyz="1 0 0"/>
-    <origin xyz="0 0 0" rpy="0 0 0"/>
+    <origin xyz="0 0 0.032" rpy="0 0 0"/>
     <limit effort="1000.0" lower="-1" upper="1" velocity="0.5"/>
   </joint>
@@ -139,5 +139,5 @@
     <child link="${prefix}z_column"/>
     <axis xyz="0 1 0"/>
-    <origin xyz="0.03005 -0.0198 0.05" rpy="0 0 0"/>
+    <origin xyz="-0.1005 0 0.0157" rpy="0 0 0"/>
     <limit effort="1000.0" lower="0" upper="0" velocity="0.5"/>
   </joint>

File: pf400_description/urdf/pf400_robot.xacro (robot description, xacro)
@@ -9,5 +9,5 @@
   </material>
   <!-- PF400 -->
-  <xacro:include filename="$(find pf400_description)/urdf/test.urdf.xacro" />
+  <xacro:include filename="$(find pf400_description)/urdf/PF400.urdf.xacro" />
   <xacro:pf400 prefix="pf400/"/>
 </robot>
