Commit message: Adding collusion descriptions

File: pf400_description/urdf/PF400.urdf.xacro (robot description, xacro)
@@ -11,4 +11,10 @@
       <material name="white"/>
     </visual>
+    <collision>
+      <geometry>
+        <mesh filename="package://pf400_description/meshes/rail_base.STL" scale="1 1 1"/>
+      </geometry>
+      <origin xyz="0 0 0" rpy="0 0 1.5708"/>
+    </collision>
   </link>
   <link name="${prefix}rail">
@@ -20,4 +26,10 @@
       <material name="white"/>
     </visual>
+      <collision>
+      <geometry>
+        <mesh filename="package://pf400_description/meshes/rail.STL" scale="1 1 1"/>
+      </geometry>
+      <origin xyz="0 0 0" rpy="1.5708 0 1.5708"/>
+    </collision>
   </link>
   <link name="${prefix}z_column">
@@ -29,4 +41,10 @@
       <material name="white"/>
     </visual>
+      <collision>
+      <geometry>
+        <mesh filename="package://pf400_description/meshes/PF400_Z_Column.STL" scale="0.001 0.001 0.00132"/>
+      </geometry>
+      <origin xyz="0 0 0.074" rpy="0 0 0"/>
+    </collision>
   </link>
   <link name="${prefix}z_carriage">
@@ -38,4 +56,10 @@
       <material name="white"/>
     </visual>
+      <collision>
+      <geometry>
+        <mesh filename="package://pf400_description/meshes/PF400_Z_Carriage.STL" scale="0.001 0.001 0.001"/>
+      </geometry>
+      <origin xyz="0 0 0.074" rpy="0 0 0"/>
+    </collision>
   </link>
   <link name="${prefix}inner_link">
@@ -47,4 +71,10 @@
       <material name="white"/>
     </visual>
+      <collision>
+      <geometry>
+        <mesh filename="package://pf400_description/meshes/PF400_Inner_Link.STL" scale="0.001 0.001 0.001"/>
+      </geometry>
+      <origin xyz="0 0 0.074" rpy="0 0 0"/>
+    </collision>
   </link>
   <link name="${prefix}outer_link">
@@ -56,4 +86,10 @@
       <material name="white"/>
     </visual>
+      <collision>
+      <geometry>
+        <mesh filename="package://pf400_description/meshes/PF400_Outer_Link.STL" scale="0.001 0.001 0.001"/>
+      </geometry>
+      <origin xyz="0 0 0.074" rpy="0 0 0"/>
+    </collision>
   </link>
   <link name="${prefix}hand">
@@ -65,4 +101,10 @@
       <material name="white"/>
     </visual>
+      <collision>
+      <geometry>
+        <mesh filename="package://pf400_description/meshes/PF400_Hand.STL" scale="0.001 0.001 0.001"/>
+      </geometry>
+      <origin xyz="0 0 0.074" rpy="0 0 0"/>
+    </collision>
   </link>
   <link name="${prefix}left_finger">
@@ -74,4 +116,10 @@
       <material name="aluminum"/>
     </visual>
+      <collision>
+      <geometry>
+        <mesh filename="package://pf400_description/meshes/pf400_left_finger.STL" scale="0.001 0.001 0.001"/>
+      </geometry>
+      <origin xyz="-0.02 -0.053 0.053" rpy="0 0 0"/>
+    </collision>
   </link>
   <link name="${prefix}right_finger">
@@ -83,4 +131,10 @@
       <material name="aluminum"/>
     </visual>
+    <collision>
+      <geometry>
+        <mesh filename="package://pf400_description/meshes/pf400_right_finger.STL" scale="0.001 0.001 0.001"/>
+      </geometry>
+      <origin xyz="-0.021 -0.028 0.105" rpy="-1.5708 0 0"/>
+    </collision>
   </link>
   <!-- Joints -->

File: pf400_description/urdf/module_carts.urdf.xacro (robot description, xacro)
@@ -11,4 +11,10 @@
       <material name="darkbluegreen"/>
     </visual>
+    <collision>
+      <geometry>
+        <mesh filename="package://pf400_description/meshes/module_cart.stl" scale="1 1 1"/>
+      </geometry>
+      <origin xyz="0 0 0" rpy="0 0 0"/>
+    </collision>
   </link>
   <link name="${prefix}cart_2">
@@ -20,4 +26,10 @@
       <material name="darkbluegreen"/>
     </visual>
+    <collision>
+      <geometry>
+        <mesh filename="package://pf400_description/meshes/module_cart.stl" scale="1 1 1"/>
+      </geometry>
+      <origin xyz="0 0 0" rpy="0 0 0"/>
+    </collision>
   </link>
   <link name="${prefix}cart_3">
@@ -29,4 +41,10 @@
       <material name="darkbluegreen"/>
     </visual>
+    <collision>
+      <geometry>
+        <mesh filename="package://pf400_description/meshes/module_cart.stl" scale="1 1 1"/>
+      </geometry>
+      <origin xyz="0 0 0" rpy="0 0 0"/>
+    </collision>
   </link>
   <link name="${prefix}cart_4">
@@ -38,4 +56,10 @@
       <material name="darkbluegreen"/>
     </visual>
+    <collision>
+      <geometry>
+        <mesh filename="package://pf400_description/meshes/module_cart.stl" scale="1 1 1"/>
+      </geometry>
+      <origin xyz="0 0 0" rpy="0 0 0"/>
+    </collision>
   </link>
   <link name="${prefix}cart_5">
@@ -47,4 +71,10 @@
       <material name="darkbluegreen"/>
     </visual>
+    <collision>
+      <geometry>
+        <mesh filename="package://pf400_description/meshes/module_cart.stl" scale="1 1 1"/>
+      </geometry>
+      <origin xyz="0 0 0" rpy="0 0 0"/>
+    </collision>
   </link>
   <link name="${prefix}cart_6">
@@ -56,4 +86,10 @@
       <material name="darkbluegreen"/>
     </visual>
+    <collision>
+      <geometry>
+        <mesh filename="package://pf400_description/meshes/module_cart.stl" scale="1 1 1"/>
+      </geometry>
+      <origin xyz="0 0 0" rpy="0 0 0"/>
+    </collision>
   </link>
   <link name="${prefix}cart_7">
@@ -65,4 +101,10 @@
       <material name="darkbluegreen"/>
     </visual>
+    <collision>
+      <geometry>
+        <mesh filename="package://pf400_description/meshes/module_cart.stl" scale="1 1 1"/>
+      </geometry>
+      <origin xyz="0 0 0" rpy="0 0 0"/>
+    </collision>
   </link>
   <link name="${prefix}cart_8">
@@ -74,4 +116,10 @@
       <material name="darkbluegreen"/>
     </visual>
+    <collision>
+      <geometry>
+        <mesh filename="package://pf400_description/meshes/module_cart.stl" scale="1 1 1"/>
+      </geometry>
+      <origin xyz="0 0 0" rpy="0 0 0"/>
+    </collision>
   </link>
   <link name="${prefix}pf400_cart">
@@ -83,4 +131,10 @@
       <material name="darkbluegreen"/>
     </visual>
+    <collision>
+      <geometry>
+        <mesh filename="package://pf400_description/meshes/PF400_module.STL" scale="0.001 0.001 0.001"/>
+      </geometry>
+      <origin xyz="-1.63 2.347 -1.11" rpy="1.5708 0 0"/>
+    </collision>
   </link>
   <!-- Joints -->

File: pf400_description/urdf/peeler.urdf.xacro (robot description, xacro)
@@ -11,4 +11,10 @@
       <material name="light_blue"/>
     </visual>
+    <collision>
+      <geometry>
+        <mesh filename="package://pf400_description/meshes/peeler_base.STL" scale="0.001 0.001 0.001"/>
+      </geometry>
+      <origin xyz="0 0 0" rpy="1.5708 0 0"/>
+    </collision>
   </link>
   <link name="${prefix}peeler_plate">
@@ -20,4 +26,10 @@
       <material name="white"/>
     </visual>
+    <collision>
+      <geometry>
+        <mesh filename="package://pf400_description/meshes/peeler_plate.STL" scale="0.001 0.001 0.001"/>
+      </geometry>
+      <origin xyz="0 0 0" rpy="0 1.5708 0"/>
+    </collision>
   </link>
   <!-- Joints -->

File: pf400_description/urdf/sealer.urdf.xacro (robot description, xacro)
@@ -11,4 +11,10 @@
       <material name="pink"/>
     </visual>
+    <collision>
+      <geometry>
+        <mesh filename="package://pf400_description/meshes/sealer_base.STL" scale="0.001 0.001 0.001"/>
+      </geometry>
+      <origin xyz="0 0 0" rpy="1.5708 0 1.5708"/>
+    </collision>
   </link>
   <link name="${prefix}sealer_plate">
@@ -20,4 +26,10 @@
       <material name="aluminum"/>
     </visual>
+    <collision>
+      <geometry>
+        <mesh filename="package://pf400_description/meshes/sealer_plate.STL" scale="0.001 0.001 0.001"/>
+      </geometry>
+      <origin xyz="0 0 0" rpy="0 1.5708 0"/>
+    </collision>
   </link>
   <!-- Joints -->

File: pf400_description/urdf/thermocycler.urdf.xacro (robot description, xacro)
@@ -11,4 +11,10 @@
       <material name="light_grey"/>
     </visual>
+    <collision>
+      <geometry>
+        <mesh filename="package://pf400_description/meshes/thermocycler_base.STL" scale="0.001 0.001 0.001"/>
+      </geometry>
+      <origin xyz="0 0.5 1.042" rpy="1.5708 0 0"/>
+    </collision>
   </link>
   <link name="${prefix}thermocycler_cap">
@@ -20,4 +26,10 @@
       <material name="red"/>
     </visual>
+    <collision>
+      <geometry>
+        <mesh filename="package://pf400_description/meshes/thermocycler_cap.STL" scale="0.001 0.001 0.001"/>
+      </geometry>
+      <origin xyz="0 0 0" rpy="0 0 0"/>
+    </collision>
   </link>
   <link name="${prefix}thermocycler_base2">
@@ -29,4 +41,10 @@
       <material name="light_grey"/>
     </visual>
+    <collision>
+      <geometry>
+        <mesh filename="package://pf400_description/meshes/thermocycler_base.STL" scale="0.001 0.001 0.001"/>
+      </geometry>
+      <origin xyz="0 0.5 1.042" rpy="1.5708 0 0"/>
+    </collision>
   </link>
   <link name="${prefix}thermocycler_cap2">
@@ -38,4 +56,10 @@
       <material name="red"/>
     </visual>
+    <collision>
+      <geometry>
+        <mesh filename="package://pf400_description/meshes/thermocycler_cap.STL" scale="0.001 0.001 0.001"/>
+      </geometry>
+      <origin xyz="0 0 0" rpy="0 0 0"/>
+    </collision>
   </link>
   <!-- Joints -->

Commit message: Changing gripper location

File: pf400_description/urdf/PF400.urdf.xacro (robot description, xacro)
@@ -110,5 +110,5 @@
   <link name="${prefix}left_finger">
     <visual>
-      <origin xyz="-0.02 -0.053 0.053" rpy="0 0 0"/>
+      <origin xyz="-0.02 -0.053 0.040" rpy="0 0 0"/>
       <geometry>
         <mesh filename="package://pf400_description/meshes/pf400_left_finger.STL" scale="0.001 0.001 0.001"/>
@@ -120,10 +120,10 @@
         <mesh filename="package://pf400_description/meshes/pf400_left_finger.STL" scale="0.001 0.001 0.001"/>
       </geometry>
-      <origin xyz="-0.02 -0.053 0.053" rpy="0 0 0"/>
+      <origin xyz="-0.02 -0.053 0.040" rpy="0 0 0"/>
     </collision>
   </link>
   <link name="${prefix}right_finger">
     <visual>
-      <origin xyz="-0.021 -0.028 0.105" rpy="-1.5708 0 0"/>
+      <origin xyz="-0.021 -0.028 0.092" rpy="-1.5708 0 0"/>
       <geometry>
         <mesh filename="package://pf400_description/meshes/pf400_right_finger.STL" scale="0.001 0.001 0.001"/>
@@ -135,5 +135,5 @@
         <mesh filename="package://pf400_description/meshes/pf400_right_finger.STL" scale="0.001 0.001 0.001"/>
       </geometry>
-      <origin xyz="-0.021 -0.028 0.105" rpy="-1.5708 0 0"/>
+      <origin xyz="-0.021 -0.028 0.092" rpy="-1.5708 0 0"/>
     </collision>
   </link>
