Commit message: Created a new module carts and materials xacro

File: pf400_description/urdf/module_carts.urdf.xacro (robot description, xacro)
@@ -1,142 +1,142 @@
 <?xml version="1.0"?>
-<robot name="PF400_Robot" xmlns:xacro="http://www.ros.org/wiki/xacro">
+<robot name="Module_Carts" xmlns:xacro="http://www.ros.org/wiki/xacro">
   <!-- Links -->
-  <xacro:macro name="pf400" params = "prefix">
-  <link name="${prefix}rail_base">
+  <xacro:macro name="Module_Carts" params = "prefix">
+  <link name="${prefix}cart_1">
     <visual>
-      <origin xyz="0.125 -0.0198 0" rpy="0 0 1.5708"/>
+      <origin xyz="1.32 0.847 0" rpy="0 0 0"/>
       <geometry>
-        <mesh filename="package://pf400_description/meshes/rail_base.STL" scale="1 1 1"/>
+        <mesh filename="package://pf400_description/meshes/module_cart.stl" scale="1 1 1"/>
       </geometry>
-      <material name="white"/>
+      <material name="darkbluegreen"/>
     </visual>
   </link>
-  <link name="${prefix}rail">
+  <link name="${prefix}cart_2">
     <visual>
-      <origin xyz="0.1309 -0.0198 0.0320" rpy="1.5708 0 1.5708"/>
+      <origin xyz="0.51 0.847 0" rpy="0 0 0"/>
       <geometry>
-        <mesh filename="package://pf400_description/meshes/rail.STL" scale="1 1 1"/>
+        <mesh filename="package://pf400_description/meshes/module_cart.stl" scale="1 1 1"/>
       </geometry>
-      <material name="white"/>
+      <material name="darkbluegreen"/>
     </visual>
   </link>
-  <link name="${prefix}z_column">
+  <link name="${prefix}cart_3">
     <visual>
-      <origin xyz="0 0 0.074" rpy="0 0 0"/>
+      <origin xyz="-0.368 0.847 0" rpy="0 0 0"/>
       <geometry>
-        <mesh filename="package://pf400_description/meshes/PF400_Z_Column.STL" scale="0.001 0.001 0.00132"/>
+        <mesh filename="package://pf400_description/meshes/module_cart.stl" scale="1 1 1"/>
       </geometry>
-      <material name="white"/>
+      <material name="darkbluegreen"/>
     </visual>
   </link>
-  <link name="${prefix}z_carriage">
+  <link name="${prefix}cart_4">
     <visual>
-      <origin xyz="0 0 0.074" rpy="0 0 0"/>
+      <origin xyz="-1.18 0.847 0" rpy="0 0 0"/>
       <geometry>
-        <mesh filename="package://pf400_description/meshes/PF400_Z_Carriage.STL" scale="0.001 0.001 0.001"/>
+        <mesh filename="package://pf400_description/meshes/module_cart.stl" scale="1 1 1"/>
       </geometry>
-      <material name="white"/>
+      <material name="darkbluegreen"/>
     </visual>
   </link>
-  <link name="${prefix}inner_link">
+  <link name="${prefix}cart_5">
     <visual>
-      <origin xyz="0 0 0.074" rpy="0 0 0"/>
+      <origin xyz="1.32  -0.548 0" rpy="0 0 0"/>
       <geometry>
-        <mesh filename="package://pf400_description/meshes/PF400_Inner_Link.STL" scale="0.001 0.001 0.001"/>
+        <mesh filename="package://pf400_description/meshes/module_cart.stl" scale="1 1 1"/>
       </geometry>
-      <material name="white"/>
+      <material name="darkbluegreen"/>
     </visual>
   </link>
-  <link name="${prefix}outer_link">
+  <link name="${prefix}cart_6">
     <visual>
-      <origin xyz="0 0 0.074" rpy="0 0 0"/>
+      <origin xyz="0.51 -0.548 0" rpy="0 0 0"/>
       <geometry>
-        <mesh filename="package://pf400_description/meshes/PF400_Outer_Link.STL" scale="0.001 0.001 0.001"/>
+        <mesh filename="package://pf400_description/meshes/module_cart.stl" scale="1 1 1"/>
       </geometry>
-      <material name="white"/>
+      <material name="darkbluegreen"/>
     </visual>
   </link>
-  <link name="${prefix}hand">
+  <link name="${prefix}cart_7">
     <visual>
-      <origin xyz="0 0 0.074" rpy="0 0 0"/>
+      <origin xyz="-0.368 -0.548 0" rpy="0 0 0"/>
       <geometry>
-        <mesh filename="package://pf400_description/meshes/PF400_Hand.STL" scale="0.001 0.001 0.001"/>
+        <mesh filename="package://pf400_description/meshes/module_cart.stl" scale="1 1 1"/>
       </geometry>
-      <material name="white"/>
+      <material name="darkbluegreen"/>
     </visual>
   </link>
-  <link name="${prefix}left_finger">
+  <link name="${prefix}cart_8">
     <visual>
-      <origin xyz="-0.02 -0.053 0.053" rpy="0 0 0"/>
+      <origin xyz="-1.18 -0.548 0" rpy="0 0 0"/>
       <geometry>
-        <mesh filename="package://pf400_description/meshes/pf400_left_finger.STL" scale="0.001 0.001 0.001"/>
+        <mesh filename="package://pf400_description/meshes/module_cart.stl" scale="1 1 1"/>
       </geometry>
-      <material name="aluminum"/>
+      <material name="darkbluegreen"/>
     </visual>
   </link>
-  <link name="${prefix}right_finger">
+  <link name="${prefix}pf400_cart">
     <visual>
-      <origin xyz="-0.021 -0.028 0.105" rpy="-1.5708 0 0"/>
+      <origin xyz="-1.63 2.347 -1.11" rpy="1.5708 0 0"/>
       <geometry>
-        <mesh filename="package://pf400_description/meshes/pf400_right_finger.STL" scale="0.001 0.001 0.001"/>
+        <mesh filename="package://pf400_description/meshes/PF400_module.STL" scale="0.001 0.001 0.001"/>
       </geometry>
-      <material name="aluminum"/>
+      <material name="darkbluegreen"/>
     </visual>
   </link>
   <!-- Joints -->
-  <joint name="J1" type="prismatic">
-    <parent link="${prefix}z_column"/>
-    <child link="${prefix}z_carriage"/>
+  <joint name="pf400_cart_to_cart_1" type="fixed">
+    <parent link="${prefix}cart_1"/>
+    <child link="${prefix}pf400_cart"/>
     <axis xyz="0 0 1"/>
-    <origin xyz="0.03005 -0.0198 0.17535" rpy="0 0 0"/>
-    <limit effort="1000.0" lower="0.002" upper="1.160" velocity="0.5"/>  </joint>
-  <joint name="J2" type="revolute">
-    <parent link="${prefix}z_carriage"/>
-    <child link="${prefix}inner_link"/>
+    <origin xyz="0 0 0" rpy="0 0 0"/>
+    <limit effort="1000.0" lower="0" upper="0" velocity="0.5"/>
+  </joint>
+  <joint name="cart_1_to_cart_2" type="fixed">
+    <parent link="${prefix}cart_2"/>
+    <child link="${prefix}cart_1"/>
     <axis xyz="0 0 1"/>
-    <origin xyz="0.173001 0.020 0.0235" rpy="0 0 0"/>
-    <limit effort="1000.0" lower="-1.62316" upper="1.62316" velocity="0.5"/>
+    <origin xyz="0 0 0" rpy="0 0 0"/>
+    <limit effort="1000.0" lower="0" upper="0" velocity="0.5"/>
   </joint>
-  <joint name="J3" type="revolute">
-    <parent link="${prefix}inner_link"/>
-    <child link="${prefix}outer_link"/>
+  <joint name="cart_2_to_cart_3" type="fixed">
+    <parent link="${prefix}cart_3"/>
+    <child link="${prefix}cart_2"/>
     <axis xyz="0 0 1"/>
-    <origin xyz="0.302 0 -0.072285" rpy="0 0 0"/>
-    <limit effort="1000.0" lower="0.175" upper="6.1" velocity="0.5"/>
+    <origin xyz="0 0 0" rpy="0 0 0"/>
+    <limit effort="1000.0" lower="0" upper="0" velocity="0.5"/>
   </joint>
-  <joint name="J4" type="revolute">
-    <parent link="${prefix}outer_link"/>
-    <child link="${prefix}hand"/>
+  <joint name="cart_3_to_cart_4" type="fixed">
+    <parent link="${prefix}cart_4"/>
+    <child link="${prefix}cart_3"/>
     <axis xyz="0 0 1"/>
-    <origin xyz="0.289 0 -0.032942" rpy="0 0 0"/>
-    <limit effort="1000.0" lower="-16.7552" upper="16.7552" velocity="0.5"/>
+    <origin xyz="0 0 0" rpy="0 0 0"/>
+    <limit effort="1000.0" lower="0" upper="0" velocity="0.5"/>
   </joint>
-  <joint name="J5" type="prismatic">
-    <parent link="${prefix}hand"/>
-    <child link="${prefix}left_finger"/>
-    <axis xyz="0 1 0"/>
-    <origin xyz="0.078573 0 -0.04269" rpy="0 0 0"/>
-    <limit effort="1000.0" lower="0.067454" upper="0.070" velocity="0.5"/>
+  <joint name="cart_4_to_cart_5" type="fixed">
+    <parent link="${prefix}cart_5"/>
+    <child link="${prefix}cart_4"/>
+    <axis xyz="0 0 1"/>
+    <origin xyz="0 0 0" rpy="0 0 0"/>
+    <limit effort="1000.0" lower="0" upper="0" velocity="0.5"/>
   </joint>
-  <joint name="J5_mirror" type="prismatic">
-    <parent link="${prefix}hand"/>
-    <child link="${prefix}right_finger"/>
-    <axis xyz="0 -1 0"/>
-    <origin xyz="0.078573 0 -0.04269" rpy="0 0 0"/>
-    <limit effort="1000.0" lower="0.067454" upper="0.070" velocity="0.5"/>
-    <mimic joint="J5" multiplier="1"/>
+  <joint name="cart_5_to_cart_6" type="fixed">
+    <parent link="${prefix}cart_6"/>
+    <child link="${prefix}cart_5"/>
+    <axis xyz="0 0 1"/>
+    <origin xyz="0 0 0" rpy="0 0 0"/>
+    <limit effort="1000.0" lower="0" upper="0" velocity="0.5"/>
   </joint>
-  <joint name="J6" type="prismatic">
-    <parent link="${prefix}rail_base"/>
-    <child link="${prefix}rail"/>
-    <axis xyz="1 0 0"/>
+  <joint name="cart_6_to_cart_7" type="fixed">
+    <parent link="${prefix}cart_7"/>
+    <child link="${prefix}cart_6"/>
+    <axis xyz="0 0 1"/>
     <origin xyz="0 0 0" rpy="0 0 0"/>
-    <limit effort="1000.0" lower="-1" upper="1" velocity="0.5"/>
+    <limit effort="1000.0" lower="0" upper="0" velocity="0.5"/>
   </joint>
-  <joint name="rail_link" type="fixed">
-    <parent link="${prefix}rail"/>
-    <child link="${prefix}z_column"/>
-    <axis xyz="0 1 0"/>
-    <origin xyz="0.03005 -0.0198 0.05" rpy="0 0 0"/>
+  <joint name="cart_7_to_cart_8" type="fixed">
+    <parent link="${prefix}cart_8"/>
+    <child link="${prefix}cart_7"/>
+    <axis xyz="0 0 1"/>
+    <origin xyz="0 0 0" rpy="0 0 0"/>
     <limit effort="1000.0" lower="0" upper="0" velocity="0.5"/>
   </joint>

File: pf400_description/urdf/pcr_workcell.urdf.xacro (robot description, xacro)
@@ -2,40 +2,5 @@
 <robot name="PCR Workcell" xmlns:xacro="http://www.ros.org/wiki/xacro">
   <!-- Materials -->
-  <material name="white">
-    <color rgba="1 1 1 1"/>
-  </material>
-  <material name="black">
-    <color rgba="0.2 0.2 0.2 1"/>
-  </material>
-  <material name="blue">
-    <color rgba="0 0 0.8 1"/>
-  </material>
-  <material name="red">
-    <color rgba="0.8 0.2 0.2 1"/>
-  </material>
-  <material name="pink">
-    <color rgba="0.6 0.4 0.6 1"/>
-  </material>
-  <material name="dark_grey">
-    <color rgba="0.4 0.4 0.4 1"/>
-  </material>
-  <material name="light_grey">
-    <color rgba="0.9 0.9 0.9 1"/>
-  </material>
-  <material name="dark_blue">
-    <color rgba="0.011764705882352941 0.027450980392156862 0.29215686274509803 1.0"/>
-  </material>
-  <material name="light_blue">
-    <color rgba="0 0.5 0.8 1.0"/>
-  </material>
-  <material name="darkbluegrey" >
-    <color rgba="0.12156862745098039 0.23137254901960785 0.30196078431372547 1.0" />
-  </material>
-  <material name="darkbluegreen" >
-    <color rgba="0.0 0.1 0.13 1.0" />
-  </material>
-  <material name="aluminum">
-    <color rgba="0.6 0.6 0.6 1"/>
-  </material>
+  <xacro:include filename="$(find pf400_description)/urdf/PF400.urdf.xacro" />
   <!-- PF400 -->
   <xacro:include filename="$(find pf400_description)/urdf/PF400.urdf.xacro" />
@@ -53,4 +18,7 @@
   <xacro:include filename="$(find pf400_description)/urdf/thermocycler.urdf.xacro" />
   <xacro:Thermocycler prefix="thermocycler/"/>
+  <!-- Module Carts -->
+  <xacro:include filename="$(find pf400_description)/urdf/module_carts.urdf.xacro" />
+  <xacro:Module_Carts prefix="module_carts/"/>
   <!-- Links -->
   <link name="OT2_2">
@@ -63,88 +31,7 @@
     </visual>
   </link>
-  <link name="module_cart_link_1">
-    <visual>
-      <origin xyz="1.32 0.847 0" rpy="0 0 0"/>
-      <geometry>
-        <mesh filename="package://pf400_description/meshes/module_cart.stl" scale="1 1 1"/>
-      </geometry>
-      <material name="darkbluegreen"/>
-    </visual>
-  </link>
-  <link name="module_cart_link_2">
-    <visual>
-      <origin xyz="0.51 0.847 0" rpy="0 0 0"/>
-      <geometry>
-        <mesh filename="package://pf400_description/meshes/module_cart.stl" scale="1 1 1"/>
-      </geometry>
-      <material name="darkbluegreen"/>
-    </visual>
-  </link>
-  <link name="module_cart_link_3">
-    <visual>
-      <origin xyz="-0.368 0.847 0" rpy="0 0 0"/>
-      <geometry>
-        <mesh filename="package://pf400_description/meshes/module_cart.stl" scale="1 1 1"/>
-      </geometry>
-      <material name="darkbluegreen"/>
-    </visual>
-  </link>
-  <link name="module_cart_link_4">
-    <visual>
-      <origin xyz="-1.18 0.847 0" rpy="0 0 0"/>
-      <geometry>
-        <mesh filename="package://pf400_description/meshes/module_cart.stl" scale="1 1 1"/>
-      </geometry>
-      <material name="darkbluegreen"/>
-    </visual>
-  </link>
-  <link name="module_cart_link_5">
-    <visual>
-      <origin xyz="1.32  -0.548 0" rpy="0 0 0"/>
-      <geometry>
-        <mesh filename="package://pf400_description/meshes/module_cart.stl" scale="1 1 1"/>
-      </geometry>
-      <material name="darkbluegreen"/>
-    </visual>
-  </link>
-  <link name="module_cart_link_6">
-    <visual>
-      <origin xyz="0.51 -0.548 0" rpy="0 0 0"/>
-      <geometry>
-        <mesh filename="package://pf400_description/meshes/module_cart.stl" scale="1 1 1"/>
-      </geometry>
-      <material name="darkbluegreen"/>
-    </visual>
-  </link>
-  <link name="module_cart_link_7">
-    <visual>
-      <origin xyz="-0.368 -0.548 0" rpy="0 0 0"/>
-      <geometry>
-        <mesh filename="package://pf400_description/meshes/module_cart.stl" scale="1 1 1"/>
-      </geometry>
-      <material name="darkbluegreen"/>
-    </visual>
-  </link>
-  <link name="module_cart_link_8">
-    <visual>
-      <origin xyz="-1.18 -0.548 0" rpy="0 0 0"/>
-      <geometry>
-        <mesh filename="package://pf400_description/meshes/module_cart.stl" scale="1 1 1"/>
-      </geometry>
-      <material name="darkbluegreen"/>
-    </visual>
-  </link>
-  <link name="pf400_module">
-    <visual>
-      <origin xyz="-1.63 2.347 -1.11" rpy="1.5708 0 0"/>
-      <geometry>
-        <mesh filename="package://pf400_description/meshes/PF400_module.STL" scale="0.001 0.001 0.001"/>
-      </geometry>
-      <material name="darkbluegreen"/>
-    </visual>
-  </link>
   <!-- Joints -->
-  <joint name="module_table" type="fixed">
-    <parent link="pf400_module"/>
+  <joint name="pf400_module" type="fixed">
+    <parent link="module_carts/pf400_cart"/>
     <child link="pf400/rail_base"/>
     <axis xyz="0 0 1"/>
@@ -152,62 +39,6 @@
     <limit effort="1000.0" lower="0" upper="0" velocity="0.5"/>
   </joint>
-  <joint name="module_cart_link_1" type="fixed">
-    <parent link="module_cart_link_1"/>
-    <child link="pf400_module"/>
-    <axis xyz="0 0 1"/>
-    <origin xyz="0 0 0" rpy="0 0 0"/>
-    <limit effort="1000.0" lower="0" upper="0" velocity="0.5"/>
-  </joint>
-  <joint name="module_cart_link_2" type="fixed">
-    <parent link="module_cart_link_2"/>
-    <child link="module_cart_link_1"/>
-    <axis xyz="0 0 1"/>
-    <origin xyz="0 0 0" rpy="0 0 0"/>
-    <limit effort="1000.0" lower="0" upper="0" velocity="0.5"/>
-  </joint>
-  <joint name="module_cart_link_3" type="fixed">
-    <parent link="module_cart_link_3"/>
-    <child link="module_cart_link_2"/>
-    <axis xyz="0 0 1"/>
-    <origin xyz="0 0 0" rpy="0 0 0"/>
-    <limit effort="1000.0" lower="0" upper="0" velocity="0.5"/>
-  </joint>
-  <joint name="module_cart_link_4" type="fixed">
-    <parent link="module_cart_link_4"/>
-    <child link="module_cart_link_3"/>
-    <axis xyz="0 0 1"/>
-    <origin xyz="0 0 0" rpy="0 0 0"/>
-    <limit effort="1000.0" lower="0" upper="0" velocity="0.5"/>
-  </joint>
-  <joint name="module_cart_link_5" type="fixed">
-    <parent link="module_cart_link_5"/>
-    <child link="module_cart_link_4"/>
-    <axis xyz="0 0 1"/>
-    <origin xyz="0 0 0" rpy="0 0 0"/>
-    <limit effort="1000.0" lower="0" upper="0" velocity="0.5"/>
-  </joint>
-  <joint name="module_cart_link_6" type="fixed">
-    <parent link="module_cart_link_6"/>
-    <child link="module_cart_link_5"/>
-    <axis xyz="0 0 1"/>
-    <origin xyz="0 0 0" rpy="0 0 0"/>
-    <limit effort="1000.0" lower="0" upper="0" velocity="0.5"/>
-  </joint>
-  <joint name="module_cart_link_7" type="fixed">
-    <parent link="module_cart_link_7"/>
-    <child link="module_cart_link_6"/>
-    <axis xyz="0 0 1"/>
-    <origin xyz="0 0 0" rpy="0 0 0"/>
-    <limit effort="1000.0" lower="0" upper="0" velocity="0.5"/>
-  </joint>
-  <joint name="module_cart_link_8" type="fixed">
-    <parent link="module_cart_link_8"/>
-    <child link="module_cart_link_7"/>
-    <axis xyz="0 0 1"/>
-    <origin xyz="0 0 0" rpy="0 0 0"/>
-    <limit effort="1000.0" lower="0" upper="0" velocity="0.5"/>
-  </joint>
   <joint name="Thermocycler_Base" type="fixed">
-    <parent link="module_cart_link_4"/>
+    <parent link="module_carts/cart_4"/>
     <child link="thermocycler/Thermocycler_Base"/>
     <axis xyz="0 0 1"/>
@@ -216,5 +47,5 @@
   </joint>
   <joint name="Peeler_Base" type="fixed">
-    <parent link="module_cart_link_5"/>
+    <parent link="module_carts/cart_5"/>
     <child link="peeler/peeler_base"/>
     <axis xyz="0 0 0"/>
@@ -223,5 +54,5 @@
   </joint>
   <joint name="Sealer_Base" type="fixed">
-    <parent link="module_cart_link_5"/>
+    <parent link="module_carts/cart_5"/>
     <child link="sealer/sealer_base"/>
     <axis xyz="0 0 1"/>
@@ -230,5 +61,5 @@
   </joint>
   <joint name="OT2" type="fixed">
-    <parent link="module_cart_link_2"/>
+    <parent link="module_carts/cart_2"/>
     <child link="ot2/OT2"/>
     <axis xyz="0 0 1"/>

Commit message: Added new pf400 table mesh

File: pf400_description/urdf/module_carts.urdf.xacro (robot description, xacro)
@@ -127,5 +127,5 @@
       <origin xyz="-1.63 2.347 -1.11" rpy="1.5708 0 0"/>
       <geometry>
-        <mesh filename="package://pf400_description/meshes/PF400_module.STL" scale="0.001 0.001 0.001"/>
+        <mesh filename="package://pf400_description/meshes/pf400_table.STL" scale="0.001 0.001 0.001"/>
       </geometry>
       <material name="darkbluegreen"/>
@@ -133,5 +133,5 @@
     <collision>
       <geometry>
-        <mesh filename="package://pf400_description/meshes/PF400_module.STL" scale="0.001 0.001 0.001"/>
+        <mesh filename="package://pf400_description/meshes/pf400_table.STL" scale="0.001 0.001 0.001"/>
       </geometry>
       <origin xyz="-1.63 2.347 -1.11" rpy="1.5708 0 0"/>

Commit message: Working on new pf400 table

File: pf400_description/urdf/module_carts.urdf.xacro (robot description, xacro)
@@ -125,5 +125,5 @@
   <link name="${prefix}pf400_cart">
     <visual>
-      <origin xyz="-1.63 2.347 -1.11" rpy="1.5708 0 0"/>
+      <origin xyz="0 0 0" rpy="1.5708 0 0"/>
       <geometry>
         <mesh filename="package://pf400_description/meshes/pf400_table.STL" scale="0.001 0.001 0.001"/>
@@ -135,5 +135,5 @@
         <mesh filename="package://pf400_description/meshes/pf400_table.STL" scale="0.001 0.001 0.001"/>
       </geometry>
-      <origin xyz="-1.63 2.347 -1.11" rpy="1.5708 0 0"/>
+      <origin xyz="0 0 0" rpy="1.5708 0 0"/>
     </collision>
   </link>

File: pf400_description/urdf/pcr_workcell.urdf.xacro (robot description, xacro)
@@ -7,15 +7,16 @@
   <xacro:pf400 prefix="pf400/"/>
   <!-- Peeler -->
-  <xacro:include filename="$(find pf400_description)/urdf/peeler.urdf.xacro" />
-  <xacro:Peeler prefix="peeler/"/>
+  <!-- <xacro:include filename="$(find pf400_description)/urdf/peeler.urdf.xacro" />
+  <xacro:Peeler prefix="peeler/"/> -->
   <!-- Sealer -->
-  <xacro:include filename="$(find pf400_description)/urdf/sealer.urdf.xacro" />
-  <xacro:Sealer prefix="sealer/"/>
+  <!-- <xacro:include filename="$(find pf400_description)/urdf/sealer.urdf.xacro" />
+  <xacro:Sealer prefix="sealer/"/> -->
   <!-- OT2 -->
-  <xacro:include filename="$(find pf400_description)/urdf/OT2.urdf.xacro" />
-  <xacro:OT2 prefix="ot2/"/>
+  <!-- <xacro:include filename="$(find pf400_description)/urdf/OT2.urdf.xacro" />
+  <xacro:OT2 prefix="ot2/"/> -->
   <!-- Thermocycler -->
-  <xacro:include filename="$(find pf400_description)/urdf/thermocycler.urdf.xacro" />
+  <!-- <xacro:include filename="$(find pf400_description)/urdf/thermocycler.urdf.xacro" />
   <xacro:Thermocycler prefix="thermocycler/"/>
+   -->
   <!-- Module Carts -->
   <xacro:include filename="$(find pf400_description)/urdf/module_carts.urdf.xacro" />
@@ -29,4 +30,5 @@
     <limit effort="1000.0" lower="0" upper="0" velocity="0.5"/>
   </joint>
+<!--
   <joint name="Thermocycler_Base" type="fixed">
     <parent link="module_carts/cart_2"/>
@@ -70,4 +72,4 @@
     <origin xyz="0.825 0.47 0" rpy="0 0 3.1416"/>
     <limit effort="1000.0" lower="0" upper="0" velocity="0.5"/>
-  </joint>
+  </joint> -->
 </robot>

Commit message: Fixewd the new table locations

File: pf400_description/urdf/module_carts.urdf.xacro (robot description, xacro)
@@ -125,5 +125,5 @@
   <link name="${prefix}pf400_cart">
     <visual>
-      <origin xyz="0 0 0" rpy="1.5708 0 0"/>
+      <origin xyz="-1.592 0.2605 -0.015" rpy="1.5708 0 0"/>
       <geometry>
         <mesh filename="package://pf400_description/meshes/pf400_table.STL" scale="0.001 0.001 0.001"/>
@@ -135,5 +135,5 @@
         <mesh filename="package://pf400_description/meshes/pf400_table.STL" scale="0.001 0.001 0.001"/>
       </geometry>
-      <origin xyz="0 0 0" rpy="1.5708 0 0"/>
+      <origin xyz="-1.592 0.261 -0.015" rpy="1.5708 0 0"/>
     </collision>
   </link>

File: pf400_description/urdf/pcr_workcell.urdf.xacro (robot description, xacro)
@@ -7,16 +7,15 @@
   <xacro:pf400 prefix="pf400/"/>
   <!-- Peeler -->
-  <!-- <xacro:include filename="$(find pf400_description)/urdf/peeler.urdf.xacro" />
-  <xacro:Peeler prefix="peeler/"/> -->
+  <xacro:include filename="$(find pf400_description)/urdf/peeler.urdf.xacro" />
+  <xacro:Peeler prefix="peeler/"/>
   <!-- Sealer -->
-  <!-- <xacro:include filename="$(find pf400_description)/urdf/sealer.urdf.xacro" />
-  <xacro:Sealer prefix="sealer/"/> -->
+  <xacro:include filename="$(find pf400_description)/urdf/sealer.urdf.xacro" />
+  <xacro:Sealer prefix="sealer/"/>
   <!-- OT2 -->
-  <!-- <xacro:include filename="$(find pf400_description)/urdf/OT2.urdf.xacro" />
-  <xacro:OT2 prefix="ot2/"/> -->
+  <xacro:include filename="$(find pf400_description)/urdf/OT2.urdf.xacro" />
+  <xacro:OT2 prefix="ot2/"/>
   <!-- Thermocycler -->
-  <!-- <xacro:include filename="$(find pf400_description)/urdf/thermocycler.urdf.xacro" />
+  <xacro:include filename="$(find pf400_description)/urdf/thermocycler.urdf.xacro" />
   <xacro:Thermocycler prefix="thermocycler/"/>
-   -->
   <!-- Module Carts -->
   <xacro:include filename="$(find pf400_description)/urdf/module_carts.urdf.xacro" />
@@ -30,5 +29,4 @@
     <limit effort="1000.0" lower="0" upper="0" velocity="0.5"/>
   </joint>
-<!--
   <joint name="Thermocycler_Base" type="fixed">
     <parent link="module_carts/cart_2"/>
@@ -72,4 +70,4 @@
     <origin xyz="0.825 0.47 0" rpy="0 0 3.1416"/>
     <limit effort="1000.0" lower="0" upper="0" velocity="0.5"/>
-  </joint> -->
+  </joint>
 </robot>
