Commit message: Fixing module locations

File: pf400_description/urdf/module_carts.urdf.xacro (robot description, xacro)
@@ -143,5 +143,5 @@
     <child link="${prefix}cart_1"/>
     <axis xyz="0 0 1"/>
-    <origin xyz="0.99 0.806 0" rpy="0 0 0"/>
+    <origin xyz="1.0 0.83 0" rpy="0 0 0"/>
     <limit effort="1000.0" lower="0" upper="0" velocity="0.5"/>
   </joint>
@@ -150,5 +150,5 @@
     <child link="${prefix}cart_2"/>
     <axis xyz="0 0 1"/>
-    <origin xyz="0.24 0.806 0" rpy="0 0 0"/>
+    <origin xyz="0.25 0.83 0" rpy="0 0 0"/>
     <limit effort="1000.0" lower="0" upper="0" velocity="0.5"/>
   </joint>
@@ -157,5 +157,5 @@
     <child link="${prefix}cart_3"/>
     <axis xyz="0 0 1"/>
-    <origin xyz="-0.51 0.806  0" rpy="0 0 0"/>
+    <origin xyz="-0.50 0.83  0" rpy="0 0 0"/>
     <limit effort="1000.0" lower="0" upper="0" velocity="0.5"/>
   </joint>
@@ -164,5 +164,5 @@
     <child link="${prefix}cart_4"/>
     <axis xyz="0 0 1"/>
-    <origin xyz="-1.26 0.806  0" rpy="0 0 0"/>
+    <origin xyz="-1.25 0.83  0" rpy="0 0 0"/>
     <limit effort="1000.0" lower="0" upper="0" velocity="0.5"/>
   </joint>
@@ -171,5 +171,5 @@
     <child link="${prefix}cart_5"/>
     <axis xyz="0 0 1"/>
-    <origin xyz="0.99 -0.451 0" rpy="0 0 0"/>
+    <origin xyz="1.00 -0.46 0" rpy="0 0 0"/>
     <limit effort="1000.0" lower="0" upper="0" velocity="0.5"/>
   </joint>
@@ -178,5 +178,5 @@
     <child link="${prefix}cart_6"/>
     <axis xyz="0 0 1"/>
-    <origin xyz="0.24 -0.451 0" rpy="0 0 0"/>
+    <origin xyz="0.25 -0.46 0" rpy="0 0 0"/>
     <limit effort="1000.0" lower="0" upper="0" velocity="0.5"/>
   </joint>
@@ -185,5 +185,5 @@
     <child link="${prefix}cart_7"/>
     <axis xyz="0 0 1"/>
-    <origin xyz="-0.51 -0.451 0" rpy="0 0 0"/>
+    <origin xyz="-0.50 -0.46 0" rpy="0 0 0"/>
     <limit effort="1000.0" lower="0" upper="0" velocity="0.5"/>
   </joint>
@@ -192,5 +192,5 @@
     <child link="${prefix}cart_8"/>
     <axis xyz="0 0 1"/>
-    <origin xyz="-1.26 -0.451 0" rpy="0 0 0"/>
+    <origin xyz="-1.25 -0.46 0" rpy="0 0 0"/>
     <limit effort="1000.0" lower="0" upper="0" velocity="0.5"/>
   </joint>

File: pf400_description/urdf/pcr_workcell.urdf.xacro (robot description, xacro)
@@ -36,5 +36,5 @@
     <child link="thermocycler/thermocycler_base"/>
     <axis xyz="0 0 0"/>
-    <origin xyz="0.2 -0.65 0" rpy="0 0 0"/>
+    <origin xyz="0.2 -0.62 0" rpy="0 0 0"/>
     <limit effort="1000.0" lower="0" upper="0" velocity="0.5"/>
   </joint>
@@ -43,5 +43,5 @@
     <child link="thermocycler/thermocycler_base2"/>
     <axis xyz="0 0 0"/>
-    <origin xyz="-0.1 -0.65 0" rpy="0 0 0"/>
+    <origin xyz="-0.1 -0.62 0" rpy="0 0 0"/>
     <limit effort="1000.0" lower="0" upper="0" velocity="0.5"/>
   </joint>
@@ -50,5 +50,5 @@
     <child link="peeler/peeler_base"/>
     <axis xyz="0 0 0"/>
-    <origin xyz="-0.17 0.19 1.042" rpy="0 0 0"/>
+    <origin xyz="-0.13 0.15 1.042" rpy="0 0 0"/>
     <limit effort="1000.0" lower="0" upper="0" velocity="0.5"/>
   </joint>
@@ -57,5 +57,5 @@
     <child link="sealer/sealer_base"/>
     <axis xyz="0 0 0"/>
-    <origin xyz="0.23 -0.51 1.042" rpy="0 0 0"/>
+    <origin xyz="0.27 -0.53 1.042" rpy="0 0 0"/>
     <limit effort="1000.0" lower="0" upper="0" velocity="0.5"/>
   </joint>

File: pf400_description/urdf/thermocycler.urdf.xacro (robot description, xacro)
@@ -68,6 +68,6 @@
     <child link="${prefix}thermocycler_cap"/>
     <axis xyz="-1 0 0"/>
-    <origin xyz="0 0.466 1.05" rpy="1.5708 0 0"/>
-    <limit effort="1000.0" lower="0" upper="1.2" velocity="0.5"/>
+    <origin xyz="0 0.466 1.05" rpy="0.4 0 0"/>
+    <limit effort="1000.0" lower="1.2" upper="1.2" velocity="0.5"/>
   </joint>
   <joint name="Thermocycler_Cap2" type="fixed">
@@ -76,5 +76,5 @@
     <axis xyz="-1 0 0"/>
     <origin xyz="0 0.466 1.05" rpy="1.5708 0 0"/>
-    <limit effort="1000.0" lower="0" upper="1.2" velocity="0.5"/>
+    <limit effort="1000.0" lower="1.2" upper="1.2" velocity="0.5"/>
   </joint>
   </xacro:macro>

Commit message: Removing extra module carts

File: pf400_description/urdf/module_carts.urdf.xacro (robot description, xacro)
@@ -3,124 +3,4 @@
   <!-- Links -->
   <xacro:macro name="Module_Carts" params = "prefix">
-  <link name="${prefix}cart_1">
-    <visual>
-      <origin xyz="0 0 0" rpy="0 0 0"/>
-      <geometry>
-        <mesh filename="package://pf400_description/meshes/module_cart.stl" scale="1 1 1"/>
-      </geometry>
-      <material name="darkbluegreen"/>
-    </visual>
-    <collision>
-      <geometry>
-        <mesh filename="package://pf400_description/meshes/module_cart.stl" scale="1 1 1"/>
-      </geometry>
-      <origin xyz="0 0 0" rpy="0 0 0"/>
-    </collision>
-  </link>
-  <link name="${prefix}cart_2">
-    <visual>
-      <origin xyz="0 0 0" rpy="0 0 0"/>
-      <geometry>
-        <mesh filename="package://pf400_description/meshes/module_cart.stl" scale="1 1 1"/>
-      </geometry>
-      <material name="darkbluegreen"/>
-    </visual>
-    <collision>
-      <geometry>
-        <mesh filename="package://pf400_description/meshes/module_cart.stl" scale="1 1 1"/>
-      </geometry>
-      <origin xyz="0 0 0" rpy="0 0 0"/>
-    </collision>
-  </link>
-  <link name="${prefix}cart_3">
-    <visual>
-      <origin xyz="0 0 0" rpy="0 0 0"/>
-      <geometry>
-        <mesh filename="package://pf400_description/meshes/module_cart.stl" scale="1 1 1"/>
-      </geometry>
-      <material name="darkbluegreen"/>
-    </visual>
-    <collision>
-      <geometry>
-        <mesh filename="package://pf400_description/meshes/module_cart.stl" scale="1 1 1"/>
-      </geometry>
-      <origin xyz="0 0 0" rpy="0 0 0"/>
-    </collision>
-  </link>
-  <link name="${prefix}cart_4">
-    <visual>
-      <origin xyz="0 0 0" rpy="0 0 0"/>
-      <geometry>
-        <mesh filename="package://pf400_description/meshes/module_cart.stl" scale="1 1 1"/>
-      </geometry>
-      <material name="darkbluegreen"/>
-    </visual>
-    <collision>
-      <geometry>
-        <mesh filename="package://pf400_description/meshes/module_cart.stl" scale="1 1 1"/>
-      </geometry>
-      <origin xyz="0 0 0" rpy="0 0 0"/>
-    </collision>
-  </link>
-  <link name="${prefix}cart_5">
-    <visual>
-      <origin xyz="0 0 0" rpy="0 0 0"/>
-      <geometry>
-        <mesh filename="package://pf400_description/meshes/module_cart.stl" scale="1 1 1"/>
-      </geometry>
-      <material name="darkbluegreen"/>
-    </visual>
-    <collision>
-      <geometry>
-        <mesh filename="package://pf400_description/meshes/module_cart.stl" scale="1 1 1"/>
-      </geometry>
-      <origin xyz="0 0 0" rpy="0 0 0"/>
-    </collision>
-  </link>
-  <link name="${prefix}cart_6">
-    <visual>
-      <origin xyz="0 0 0" rpy="0 0 0"/>
-      <geometry>
-        <mesh filename="package://pf400_description/meshes/module_cart.stl" scale="1 1 1"/>
-      </geometry>
-      <material name="darkbluegreen"/>
-    </visual>
-    <collision>
-      <geometry>
-        <mesh filename="package://pf400_description/meshes/module_cart.stl" scale="1 1 1"/>
-      </geometry>
-      <origin xyz="0 0 0" rpy="0 0 0"/>
-    </collision>
-  </link>
-  <link name="${prefix}cart_7">
-    <visual>
-      <origin xyz="0 0 0" rpy="0 0 0"/>
-      <geometry>
-        <mesh filename="package://pf400_description/meshes/module_cart.stl" scale="1 1 1"/>
-      </geometry>
-      <material name="darkbluegreen"/>
-    </visual>
-    <collision>
-      <geometry>
-        <mesh filename="package://pf400_description/meshes/module_cart.stl" scale="1 1 1"/>
-      </geometry>
-      <origin xyz="0 0 0" rpy="0 0 0"/>
-    </collision>
-  </link>
-  <link name="${prefix}cart_8">
-    <visual>
-      <origin xyz="0 0 0" rpy="0 0 0"/>
-      <geometry>
-        <mesh filename="package://pf400_description/meshes/module_cart.stl" scale="1 1 1"/>
-      </geometry>
-      <material name="darkbluegreen"/>
-    </visual>
-    <collision>
-      <geometry>
-        <mesh filename="package://pf400_description/meshes/module_cart.stl" scale="1 1 1"/>
-      </geometry>
-      <origin xyz="0 0 0" rpy="0 0 0"/>
-    </collision>
-  </link>
   <link name="${prefix}pf400_cart">
     <visual>
@@ -139,60 +19,4 @@
   </link>
   <!-- Joints -->
-  <joint name="pf400_cart_to_cart_1" type="fixed">
-    <parent link="${prefix}pf400_cart"/>
-    <child link="${prefix}cart_1"/>
-    <axis xyz="0 0 1"/>
-    <origin xyz="1.0 0.83 0" rpy="0 0 0"/>
-    <limit effort="1000.0" lower="0" upper="0" velocity="0.5"/>
-  </joint>
-  <joint name="pf400_cart_to_cart_2" type="fixed">
-    <parent link="${prefix}pf400_cart"/>
-    <child link="${prefix}cart_2"/>
-    <axis xyz="0 0 1"/>
-    <origin xyz="0.25 0.83 0" rpy="0 0 0"/>
-    <limit effort="1000.0" lower="0" upper="0" velocity="0.5"/>
-  </joint>
-  <joint name="pf400_cart_to_cart_3" type="fixed">
-    <parent link="${prefix}pf400_cart"/>
-    <child link="${prefix}cart_3"/>
-    <axis xyz="0 0 1"/>
-    <origin xyz="-0.50 0.83  0" rpy="0 0 0"/>
-    <limit effort="1000.0" lower="0" upper="0" velocity="0.5"/>
-  </joint>
-  <joint name="pf400_cart_to_cart_4" type="fixed">
-    <parent link="${prefix}pf400_cart"/>
-    <child link="${prefix}cart_4"/>
-    <axis xyz="0 0 1"/>
-    <origin xyz="-1.25 0.83  0" rpy="0 0 0"/>
-    <limit effort="1000.0" lower="0" upper="0" velocity="0.5"/>
-  </joint>
-  <joint name="pf400_cart_to_cart_5" type="fixed">
-    <parent link="${prefix}pf400_cart"/>
-    <child link="${prefix}cart_5"/>
-    <axis xyz="0 0 1"/>
-    <origin xyz="1.00 -0.46 0" rpy="0 0 0"/>
-    <limit effort="1000.0" lower="0" upper="0" velocity="0.5"/>
-  </joint>
-  <joint name="pf400_cart_to_cart_6" type="fixed">
-    <parent link="${prefix}pf400_cart"/>
-    <child link="${prefix}cart_6"/>
-    <axis xyz="0 0 1"/>
-    <origin xyz="0.25 -0.46 0" rpy="0 0 0"/>
-    <limit effort="1000.0" lower="0" upper="0" velocity="0.5"/>
-  </joint>
-  <joint name="pf400_cart_to_cart_7" type="fixed">
-    <parent link="${prefix}pf400_cart"/>
-    <child link="${prefix}cart_7"/>
-    <axis xyz="0 0 1"/>
-    <origin xyz="-0.50 -0.46 0" rpy="0 0 0"/>
-    <limit effort="1000.0" lower="0" upper="0" velocity="0.5"/>
-  </joint>
-  <joint name="pf400_cart_to_cart_8" type="fixed">
-    <parent link="${prefix}pf400_cart"/>
-    <child link="${prefix}cart_8"/>
-    <axis xyz="0 0 1"/>
-    <origin xyz="-1.25 -0.46 0" rpy="0 0 0"/>
-    <limit effort="1000.0" lower="0" upper="0" velocity="0.5"/>
-  </joint>
   </xacro:macro>
 </robot>
